Commit message: Initial commit Kinova arm

File: qm_description/urdf/quadruped/aliengo.urdf (robot description, URDF)
Before this commit: robot robot, 18 links, 17 joints
Links:
- link LF_calf: geometry collision box size=0.25 0.0208 0.016; visual mesh filename=package://qm_description/meshes/quadruped/aliengo/calf_corr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 scale=1 1 1
- link LF_hip: geometry collision cylinder length=0.0418 radius=0.046; visual mesh filename=package://qm_description/meshes/quadruped/aliengo/hip.dae scale=1 1 1
- link LF_thigh: geometry collision box size=0.25 0.0374 0.043; collision cylinder length=0.03 radius=0.044
- link LH_calf: geometry collision box size=0.25 0.0208 0.016; visual mesh filename=package://qm_description/meshes/quadruped/aliengo/calf_corr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 scale=1 1 1
- link LH_hip: geometry collision cylinder length=0.0418 radius=0.046; visual mesh filename=package://qm_description/meshes/quadruped/aliengo/hip.dae scale=1 1 1
- link LH_thigh: geometry collision box size=0.25 0.0374 0.043; collision cylinder length=0.03 radius=0.044
- link RF_calf: geometry collision box size=0.25 0.0208 0.016; visual mesh filename=package://qm_description/meshes/quadruped/aliengo/calf_corr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 scale=1 1 1
- link RF_hip: geometry collision cylinder length=0.0418 radius=0.046; visual mesh filename=package://qm_description/meshes/quadruped/aliengo/hip.dae scale=1 1 1
- link RF_thigh: geometry collision box size=0.25 0.0374 0.043; collision cylinder length=0.03 radius=0.044
- link RH_calf: geometry collision box size=0.25 0.0208 0.016; visual mesh filename=package://qm_description/meshes/quadruped/aliengo/calf_corr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 scale=1 1 1
- link RH_hip: geometry collision cylinder length=0.0418 radius=0.046; visual mesh filename=package://qm_description/meshes/quadruped/aliengo/hip.dae scale=1 1 1
- link RH_thigh: geometry collision box size=0.25 0.0374 0.043; collision cylinder length=0.03 radius=0.044
- link base: geometry collision box size=0.647 0.15 0.112; visual mesh filename=package://qm_description/meshes/quadruped/aliengo/trunk.dae scale=1 1 1

File: qm_description/urdf/quadruped/common/leg.xacro (robot description, xacro)
@@ -1,5 +1,5 @@
 <?xml version="1.0"?>
 <robot xmlns:xacro="http://www.ros.org/wiki/xacro">
-    <xacro:include filename="$(find qm_description)/urdf/qudraputed/common/transmission.xacro"/>
+    <xacro:include filename="$(find qm_description)/urdf/quadruped/common/transmission.xacro"/>
     <xacro:macro name="leg" params="prefix mirror mirror_dae front_hind front_hind_dae *origin">
         <joint name="${prefix}_HAA" type="revolute">
@@ -33,8 +33,8 @@
                 </xacro:if>
                 <geometry>
-                    <mesh filename="package://qm_description/meshes/qudraputed/$(arg robot_type)/hip.dae"
+                    <mesh filename="package://qm_description/meshes/quadruped/$(arg robot_type)/hip.dae"
                           scale="1 1 1"/>
                 </geometry>
-                <material name="orange"/>
+                <material name="black"/>
             </visual>
             <collision>
@@ -67,13 +67,13 @@
                 <geometry>
                     <xacro:if value="${mirror_dae == True}">
-                        <mesh filename="package://qm_description/meshes/qudraputed/$(arg robot_type)/thigh.dae"
+                        <mesh filename="package://qm_description/meshes/quadruped/$(arg robot_type)/thigh.dae"
                               scale="1 1 1"/>
                     </xacro:if>
                     <xacro:if value="${mirror_dae == False}">
-                        <mesh filename="package://qm_description/meshes/qudraputed/$(arg robot_type)/thigh_mirror.dae"
+                        <mesh filename="package://qm_description/meshes/quadruped/$(arg robot_type)/thigh_mirror.dae"
                               scale="1 1 1"/>
                     </xacro:if>
                 </geometry>
-                <material name="orange"/>
+                <material name="black"/>
             </visual>
             <collision>
@@ -110,8 +110,8 @@
                 <origin rpy="0 0 0" xyz="0 0 0"/>
                 <geometry>
-                    <mesh filename="package://qm_description/meshes/qudraputed/$(arg robot_type)/calf.dae"
+                    <mesh filename="package://qm_description/meshes/quadruped/$(arg robot_type)/calf_corrected.stl"
                           scale="1 1 1"/>
                 </geometry>
-                <material name="orange"/>
+                <material name="black"/>
             </visual>
             <collision>
@@ -141,5 +141,5 @@
                     <sphere radius="${foot_radius-0.01}"/>
                 </geometry>
-                <material name="orange"/>
+                <material name="black"/>
             </visual>
             <collision>

File: qm_description/urdf/quadruped_manipulator/robot.urdf (robot description, URDF)
Before this commit: robot qm, 27 links, 26 joints
Links:
- link LF_calf: geometry collision box size=0.25 0.0208 0.016; visual mesh filename=package://qm_description/meshes/quadruped/aliengo/calf_corr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 scale=1 1 1
- link LF_hip: geometry collision cylinder length=0.0418 radius=0.046; visual mesh filename=package://qm_description/meshes/quadruped/aliengo/hip.dae scale=1 1 1
- link LF_thigh: geometry collision box size=0.25 0.0374 0.043; collision cylinder length=0.03 radius=0.044
- link LH_calf: geometry collision box size=0.25 0.0208 0.016; visual mesh filename=package://qm_description/meshes/quadruped/aliengo/calf_corr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 scale=1 1 1
- link LH_hip: geometry collision cylinder length=0.0418 radius=0.046; visual mesh filename=package://qm_description/meshes/quadruped/aliengo/hip.dae scale=1 1 1
- link LH_thigh: geometry collision box size=0.25 0.0374 0.043; collision cylinder length=0.03 radius=0.044
- link RF_calf: geometry collision box size=0.25 0.0208 0.016; visual mesh filename=package://qm_description/meshes/quadruped/aliengo/calf_corr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 scale=1 1 1
- link RF_hip: geometry collision cylinder length=0.0418 radius=0.046; visual mesh filename=package://qm_description/meshes/quadruped/aliengo/hip.dae scale=1 1 1
- link RF_thigh: geometry collision box size=0.25 0.0374 0.043; collision cylinder length=0.03 radius=0.044
- link RH_calf: geometry collision box size=0.25 0.0208 0.016; visual mesh filename=package://qm_description/meshes/quadruped/aliengo/calf_corr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 scale=1 1 1
- link RH_hip: geometry collision cylinder length=0.0418 radius=0.046; visual mesh filename=package://qm_description/meshes/quadruped/aliengo/hip.dae scale=1 1 1
- link RH_thigh: geometry collision box size=0.25 0.0374 0.043; collision cylinder length=0.03 radius=0.044
- link base: geometry collision box size=0.647 0.15 0.112; visual mesh filename=package://qm_description/meshes/quadruped/aliengo/trunk.dae scale=1 1 1
