Commit message: Update URDF

File: qm_description/urdf/quadruped_manipulator/robot.urdf (robot description, URDF)
Before this commit: robot qm, 28 links, 27 joints
Links:
- removed link unitree_imu
- removed link world
- added link imu_link, mass 0.001; collision box size=.001 .001 .001; visual box size=0.001 0.001 0.001
- added link trunk, mass 11.041; collision box size=0.647 0.15 0.112; visual mesh filename=package://qm_description/meshes/quadruped/aliengo/trunk.dae scale=1 1 1
- link base: mass 11.041 -> None; geometry visual box size=0.001 0.001 0.001
Joints:
- removed joint base_static_joint
- removed joint unitree_imu_joint
- added joint floating_base: type fixed, parent base, child trunk, origin xyz=0 0 0 rpy=0 0 0
- added joint imu_joint: type fixed, parent trunk, child imu_link, origin xyz=0 0 0 rpy=0 0 0
- joint trunk_arm_joint: parent base -> trunk
