Commit message: Gazebo Z1 arm debugging

File: qm_description/urdf/quadruped_manipulator/gazebo.xacro (robot description, xacro)
@@ -57,6 +57,6 @@
     </gazebo>
     <!-- Foot contacts. -->
-    <gazebo reference="FR_calf">
-        <sensor name="FR_foot_contact" type="contact">
+    <gazebo reference="RF_calf">
+        <sensor name="RF_foot_contact" type="contact">
         <update_rate>100</update_rate>
         <plugin name="contactPlugin" filename="libunitreeFootContactPlugin.so"/>
@@ -66,6 +66,6 @@
         </sensor>
     </gazebo>
-    <gazebo reference="FL_calf">
-        <sensor name="FL_foot_contact" type="contact">
+    <gazebo reference="LF_calf">
+        <sensor name="LF_foot_contact" type="contact">
         <update_rate>100</update_rate>
         <plugin name="contactPlugin" filename="libunitreeFootContactPlugin.so"/>
@@ -75,6 +75,6 @@
         </sensor>
     </gazebo>
-    <gazebo reference="RR_calf">
-        <sensor name="RR_foot_contact" type="contact">
+    <gazebo reference="RH_calf">
+        <sensor name="RH_foot_contact" type="contact">
         <update_rate>100</update_rate>
         <plugin name="contactPlugin" filename="libunitreeFootContactPlugin.so"/>
@@ -84,6 +84,6 @@
         </sensor>
     </gazebo>
-    <gazebo reference="RL_calf">
-        <sensor name="RL_foot_contact" type="contact">
+    <gazebo reference="LH_calf">
+        <sensor name="LH_foot_contact" type="contact">
         <update_rate>100</update_rate>
         <plugin name="contactPlugin" filename="libunitreeFootContactPlugin.so"/>
@@ -94,5 +94,5 @@
     </gazebo>
     <!-- Visualization of Foot contacts. -->
-    <gazebo reference="FR_foot">
+    <gazebo reference="RF_foot">
         <visual>
             <plugin name="drawForcePlugin" filename="libunitreeDrawForcePlugin.so">
@@ -101,5 +101,5 @@
         </visual>
     </gazebo>
-    <gazebo reference="FL_foot">
+    <gazebo reference="LF_foot">
         <visual>
             <plugin name="drawForcePlugin" filename="libunitreeDrawForcePlugin.so">
@@ -108,5 +108,5 @@
         </visual>
     </gazebo>
-    <gazebo reference="RR_foot">
+    <gazebo reference="RH_foot">
         <visual>
             <plugin name="drawForcePlugin" filename="libunitreeDrawForcePlugin.so">
@@ -115,5 +115,5 @@
         </visual>
     </gazebo>
-    <gazebo reference="RL_foot">
+    <gazebo reference="LH_foot">
         <visual>
             <plugin name="drawForcePlugin" filename="libunitreeDrawForcePlugin.so">
@@ -141,97 +141,113 @@
         <material>Gazebo/Red</material>
     </gazebo>
-    <!-- FL leg -->
-    <gazebo reference="FL_hip">
-        <mu1>0.2</mu1>
-        <mu2>0.2</mu2>
-    </gazebo>
-    <gazebo reference="FL_thigh">
-        <mu1>0.2</mu1>
-        <mu2>0.2</mu2>
-        <self_collide>1</self_collide>
-        <kp  value="1000000.0"/>
-        <kd  value="1.0"/>
-    </gazebo>
-    <gazebo reference="FL_calf">
-        <mu1>0.2</mu1>
-        <mu2>0.2</mu2>
-        <self_collide>1</self_collide>
-    </gazebo>
-    <gazebo reference="FL_foot">
-        <mu1>0.6</mu1>
-        <mu2>0.6</mu2>
-        <self_collide>1</self_collide>
-        <kp  value="1000000.0"/>
-        <kd  value="1.0"/>
-    </gazebo>
-    <!-- FR leg -->
-    <gazebo reference="FR_hip">
-        <mu1>0.2</mu1>
-        <mu2>0.2</mu2>
-    </gazebo>
-    <gazebo reference="FR_thigh">
-        <mu1>0.2</mu1>
-        <mu2>0.2</mu2>
-        <self_collide>1</self_collide>
-        <kp  value="1000000.0"/>
-        <kd  value="1.0"/>
-    </gazebo>
-    <gazebo reference="FR_calf">
-        <mu1>0.2</mu1>
-        <mu2>0.2</mu2>
-        <self_collide>1</self_collide>
-    </gazebo>
-    <gazebo reference="FR_foot">
-        <mu1>0.6</mu1>
-        <mu2>0.6</mu2>
-        <self_collide>1</self_collide>
-        <kp  value="1000000.0"/>
-        <kd  value="1.0"/>
-    </gazebo>
-    <!-- RL leg -->
-    <gazebo reference="RL_hip">
-        <mu1>0.2</mu1>
-        <mu2>0.2</mu2>
-    </gazebo>
-    <gazebo reference="RL_thigh">
-        <mu1>0.2</mu1>
-        <mu2>0.2</mu2>
-        <self_collide>1</self_collide>
-        <kp  value="1000000.0"/>
-        <kd  value="1.0"/>
-    </gazebo>
-    <gazebo reference="RL_calf">
-        <mu1>0.2</mu1>
-        <mu2>0.2</mu2>
-        <self_collide>1</self_collide>
-    </gazebo>
-    <gazebo reference="RL_foot">
-        <mu1>0.6</mu1>
-        <mu2>0.6</mu2>
-        <self_collide>1</self_collide>
-        <kp  value="1000000.0"/>
-        <kd  value="1.0"/>
-    </gazebo>
-    <!-- RR leg -->
-    <gazebo reference="RR_hip">
-        <mu1>0.2</mu1>
-        <mu2>0.2</mu2>
-    </gazebo>
-    <gazebo reference="RR_thigh">
-        <mu1>0.2</mu1>
-        <mu2>0.2</mu2>
-        <self_collide>1</self_collide>
-        <kp  value="1000000.0"/>
-        <kd  value="1.0"/>
-    </gazebo>
-    <gazebo reference="RR_calf">
-        <mu1>0.2</mu1>
-        <mu2>0.2</mu2>
-        <self_collide>1</self_collide>
-    </gazebo>
-    <gazebo reference="RR_foot">
-        <mu1>0.6</mu1>
-        <mu2>0.6</mu2>
-        <self_collide>1</self_collide>
+    <!-- LF leg -->
+    <gazebo reference="LF_hip">
+        <mu1>0.2</mu1>
+        <mu2>0.2</mu2>
+        <material>Gazebo/Black</material>
+    </gazebo>
+    <gazebo reference="LF_thigh">
+        <mu1>0.2</mu1>
+        <mu2>0.2</mu2>
+        <self_collide>1</self_collide>
+        <kp  value="1000000.0"/>
+        <kd  value="1.0"/>
+        <material>Gazebo/Black</material>
+    </gazebo>
+    <gazebo reference="LF_calf">
+        <mu1>0.2</mu1>
+        <mu2>0.2</mu2>
+        <self_collide>1</self_collide>
+        <material>Gazebo/Black</material>
+    </gazebo>
+    <gazebo reference="LF_foot">
+        <mu1>0.6</mu1>
+        <mu2>0.6</mu2>
+        <self_collide>1</self_collide>
+        <kp  value="1000000.0"/>
+        <kd  value="1.0"/>
+        <material>Gazebo/Black</material>
+    </gazebo>
+    <!-- RF leg -->
+    <gazebo reference="RF_hip">
+        <mu1>0.2</mu1>
+        <mu2>0.2</mu2>
+        <material>Gazebo/Black</material>
+    </gazebo>
+    <gazebo reference="RF_thigh">
+        <mu1>0.2</mu1>
+        <mu2>0.2</mu2>
+        <self_collide>1</self_collide>
+        <kp  value="1000000.0"/>
+        <kd  value="1.0"/>
+        <material>Gazebo/Black</material>
+    </gazebo>
+    <gazebo reference="RF_calf">
+        <mu1>0.2</mu1>
+        <mu2>0.2</mu2>
+        <self_collide>1</self_collide>
+        <material>Gazebo/Black</material>
+    </gazebo>
+    <gazebo reference="RF_foot">
+        <mu1>0.6</mu1>
+        <mu2>0.6</mu2>
+        <self_collide>1</self_collide>
+        <kp  value="1000000.0"/>
+        <kd  value="1.0"/>
+        <material>Gazebo/Black</material>
+    </gazebo>
+    <!-- LH leg -->
+    <gazebo reference="LH_hip">
+        <mu1>0.2</mu1>
+        <mu2>0.2</mu2>
+        <material>Gazebo/Black</material>
+    </gazebo>
+    <gazebo reference="LH_thigh">
+        <mu1>0.2</mu1>
+        <mu2>0.2</mu2>
+        <self_collide>1</self_collide>
+        <kp  value="1000000.0"/>
+        <kd  value="1.0"/>
+        <material>Gazebo/Black</material>
+    </gazebo>
+    <gazebo reference="LH_calf">
+        <mu1>0.2</mu1>
+        <mu2>0.2</mu2>
+        <self_collide>1</self_collide>
+        <material>Gazebo/Black</material>
+    </gazebo>
+    <gazebo reference="LH_foot">
+        <mu1>0.6</mu1>
+        <mu2>0.6</mu2>
+        <self_collide>1</self_collide>
+        <kp  value="1000000.0"/>
+        <kd  value="1.0"/>
+        <material>Gazebo/Black</material>
+    </gazebo>
+    <!-- RH leg -->
+    <gazebo reference="RH_hip">
+        <mu1>0.2</mu1>
+        <mu2>0.2</mu2>
+        <material>Gazebo/Black</material>
+    </gazebo>
+    <gazebo reference="RH_thigh">
+        <mu1>0.2</mu1>
+        <mu2>0.2</mu2>
+        <self_collide>1</self_collide>
+        <kp  value="1000000.0"/>
+        <kd  value="1.0"/>
+        <material>Gazebo/Black</material>
+    </gazebo>
+    <gazebo reference="RH_calf">
+        <mu1>0.2</mu1>
+        <mu2>0.2</mu2>
+        <self_collide>1</self_collide>
+        <material>Gazebo/Black</material>
+    </gazebo>
+    <gazebo reference="RH_foot">
+        <mu1>0.6</mu1>
+        <mu2>0.6</mu2>
+        <self_collide>1</self_collide>
+        <material>Gazebo/Black</material>
         <kp  value="1000000.0"/>
         <kd  value="1.0"/>
@@ -262,22 +278,11 @@
         <material>Gazebo/Grey</material>
     </gazebo>
-    <!-- Configuration for the gripperStator link in Gazebo -->
     <gazebo reference="gripperStator">
-        <material>Gazebo/Black</material>
-        <mu1>0.5</mu1>
-        <mu2>0.5</mu2>
-    </gazebo>
-    <!-- Configuration for the jointGripper in Gazebo -->
-    <gazebo reference="jointGripper">
-        <mu1>0.2</mu1>
-        <mu2>0.2</mu2>
-        <kp>1000000.0</kp>
-        <kd>1.0</kd>
-    </gazebo>
-    <!-- Configuration for the gripperMover link in Gazebo -->
+        <self_collide>true</self_collide>
+        <material>Gazebo/Black</material>
+    </gazebo>
     <gazebo reference="gripperMover">
-        <material>Gazebo/Black</material>
-        <mu1>0.5</mu1>
-        <mu2>0.5</mu2>
+        <self_collide>true</self_collide>
+        <material>Gazebo/Black</material>
     </gazebo>
 </robot>

File: qm_description/urdf/quadruped_manipulator/robot.xacro (robot description, xacro)
@@ -10,5 +10,4 @@
     <xacro:include filename="$(find qm_description)/urdf/manipulator/const.xacro"/>
     <xacro:include filename="$(find qm_description)/urdf/manipulator/transmission.xacro"/>
-    <xacro:arg name="UnitreeGripper" default="true"/>
     <!-- Debug mode will hung up the robot, use "true" or "false" to switch it. -->
     <xacro:if value="$(arg DEBUG)">
@@ -269,68 +268,60 @@
         </inertial>
     </link>
-    <xacro:if value="$(arg UnitreeGripper)">
-        <joint name="gripperStator" type="fixed">
-            <origin rpy="0 0 0" xyz="0.051 0.0 0.0"/>
-            <parent link="link06"/>
-            <child link="gripperStator"/>
-        </joint>
-        <link name="gripperStator">
-            <visual>
-                <geometry>
-                    <mesh filename="package://qm_description/meshes/manipulator/z1_GripperStator.stl" scale="1 1 1"/>
-                </geometry>
-                <material name="grey"/>
-            </visual>
-            <collision>
-                <geometry>
-                    <mesh filename="package://qm_description/meshes/manipulator/z1_GripperStator.stl" scale="1 1 1"/>
-                </geometry>
-            </collision>
-            <inertial>
-                <origin rpy="0 0 0" xyz="${GripperStator_ComX} ${GripperStator_ComY} ${GripperStator_ComZ}"/>
-                <mass value="${GripperStator_Mass}"/>
-                <inertia
-                    ixx="${GripperStator_Ixx}" ixy="${GripperStator_Ixy}" ixz="${GripperStator_Ixz}"
-                    iyy="${GripperStator_Iyy}" iyz="${GripperStator_Iyz}"
-                    izz="${GripperStator_Izz}"/>
-            </inertial>
-        </link>
-        <joint name="jointGripper" type="revolute">
-            <origin rpy="0 0 0" xyz="0.049 0.0 0"/>
-            <parent link="gripperStator"/>
-            <child link="gripperMover"/>
-            <axis xyz="0 1 0"/>
-            <dynamics damping="${jointDamping}" friction="${jointFriction}"/>
-            <limit effort="${torqueMax}" velocity="${velocityMax}" lower="${Gripper_PositionMin}" upper="${Gripper_PositionMax}"/>
-        </joint>
-        <link name="gripperMover">
-            <visual>
-                <geometry>
-                    <mesh filename="package://qm_description/meshes/manipulator/z1_GripperMover.stl" scale="1 1 1"/>
-                </geometry>
-                <material name="grey"/>
-            </visual>
-            <collision>
-                <geometry>
-                    <mesh filename="package://qm_description/meshes/manipulator/z1_GripperMover.stl" scale="1 1 1"/>
-                </geometry>
-            </collision>
-            <inertial>
-                <origin rpy="0 0 0" xyz="${GripperMover_ComX} ${GripperMover_ComY} ${GripperMover_ComZ}"/>
-                <mass value="${GripperMover_Mass}"/>
-                <inertia
-                    ixx="${GripperMover_Ixx}" ixy="${GripperMover_Ixy}" ixz="${GripperMover_Ixz}"
-                    iyy="${GripperMover_Iyy}" iyz="${GripperMover_Iyz}"
-                    izz="${GripperMover_Izz}"/>
-            </inertial>
-        </link>
-        <xacro:motorTransmission name="Gripper"/>
-        <gazebo reference="gripperStator">
-            <self_collide>true</self_collide>
-        </gazebo>
-        <gazebo reference="gripperMover">
-            <self_collide>true</self_collide>
-        </gazebo>
-    </xacro:if>
+    <joint name="gripperStator" type="fixed">
+        <origin rpy="0 0 0" xyz="0.051 0.0 0.0"/>
+        <parent link="link06"/>
+        <child link="gripperStator"/>
+    </joint>
+    <link name="gripperStator">
+        <visual>
+            <geometry>
+                <mesh filename="package://qm_description/meshes/manipulator/z1_GripperStator.stl" scale="1 1 1"/>
+            </geometry>
+            <material name="grey"/>
+        </visual>
+        <collision>
+            <geometry>
+                <mesh filename="package://qm_description/meshes/manipulator/z1_GripperStator.stl" scale="1 1 1"/>
+            </geometry>
+        </collision>
+        <inertial>
+            <origin rpy="0 0 0" xyz="${GripperStator_ComX} ${GripperStator_ComY} ${GripperStator_ComZ}"/>
+            <mass value="${GripperStator_Mass}"/>
+            <inertia
+                ixx="${GripperStator_Ixx}" ixy="${GripperStator_Ixy}" ixz="${GripperStator_Ixz}"
+                iyy="${GripperStator_Iyy}" iyz="${GripperStator_Iyz}"
+                izz="${GripperStator_Izz}"/>
+        </inertial>
+    </link>
+    <joint name="jointGripper" type="revolute">
+        <origin rpy="0 0 0" xyz="0.049 0.0 0"/>
+        <parent link="gripperStator"/>
+        <child link="gripperMover"/>
+        <axis xyz="0 1 0"/>
+        <dynamics damping="${jointDamping}" friction="${jointFriction}"/>
+        <limit effort="${torqueMax}" velocity="${velocityMax}" lower="${Gripper_PositionMin}" upper="${Gripper_PositionMax}"/>
+    </joint>
+    <link name="gripperMover">
+        <visual>
+            <geometry>
+                <mesh filename="package://qm_description/meshes/manipulator/z1_GripperMover.stl" scale="1 1 1"/>
+            </geometry>
+            <material name="grey"/>
+        </visual>
+        <collision>
+            <geometry>
+                <mesh filename="package://qm_description/meshes/manipulator/z1_GripperMover.stl" scale="1 1 1"/>
+            </geometry>
+        </collision>
+        <inertial>
+            <origin rpy="0 0 0" xyz="${GripperMover_ComX} ${GripperMover_ComY} ${GripperMover_ComZ}"/>
+            <mass value="${GripperMover_Mass}"/>
+            <inertia
+                ixx="${GripperMover_Ixx}" ixy="${GripperMover_Ixy}" ixz="${GripperMover_Ixz}"
+                iyy="${GripperMover_Iyy}" iyz="${GripperMover_Iyz}"
+                izz="${GripperMover_Izz}"/>
+        </inertial>
+    </link>
+    <xacro:motorTransmission name="Gripper"/>
     <xacro:motorTransmission name="1"/>
     <xacro:motorTransmission name="2"/>

Commit message: Update z1_arm

File: qm_description/urdf/quadruped_manipulator/gazebo.xacro (robot description, xacro)
@@ -267,21 +267,19 @@
     </gazebo>
     <gazebo reference="link04">
+        <material>Gazebo/Grey</material>
         <self_collide>true</self_collide>
-        <material>Gazebo/Grey</material>
     </gazebo>
     <gazebo reference="link05">
+        <material>Gazebo/Grey</material>
         <self_collide>true</self_collide>
-        <material>Gazebo/Grey</material>
     </gazebo>
     <gazebo reference="link06">
+        <material>Gazebo/Grey</material>
         <self_collide>true</self_collide>
-        <material>Gazebo/Grey</material>
     </gazebo>
     <gazebo reference="gripperStator">
-        <self_collide>true</self_collide>
         <material>Gazebo/Black</material>
     </gazebo>
     <gazebo reference="gripperMover">
-        <self_collide>true</self_collide>
         <material>Gazebo/Black</material>
     </gazebo>

File: qm_description/urdf/quadruped_manipulator/robot.xacro (robot description, xacro)
@@ -255,7 +255,7 @@
         <collision>
             <geometry>
-                <cylinder length="${motor_height}" radius="${motor_diameter}"/>
-            </geometry>
-            <origin rpy="0 ${PI/2.0} 0" xyz="${motor_height/2.0} 0 0"/>
+                <cylinder length="${motor_height - 0.01}" radius="${motor_diameter}"/>
+            </geometry>
+            <origin rpy="0 ${PI/2.0} 0" xyz="${(motor_height - 0.01)/2.0} 0 0"/>
         </collision>
         <inertial>
