Commit message: Debug gazebo

File: qm_description/urdf/quadruped_manipulator/gazebo.xacro (robot description, xacro)
@@ -62,5 +62,5 @@
         <plugin name="contactPlugin" filename="libunitreeFootContactPlugin.so"/>
         <contact>
-            <collision>FR_calf_fixed_joint_lump__FR_foot_collision_1</collision>
+            <collision>RF_calf_fixed_joint_lump__RF_foot_collision_1</collision>
         </contact>
         </sensor>
@@ -71,5 +71,5 @@
         <plugin name="contactPlugin" filename="libunitreeFootContactPlugin.so"/>
         <contact>
-            <collision>FL_calf_fixed_joint_lump__FL_foot_collision_1</collision>
+            <collision>LF_calf_fixed_joint_lump__LF_foot_collision_1</collision>
         </contact>
         </sensor>
@@ -80,5 +80,5 @@
         <plugin name="contactPlugin" filename="libunitreeFootContactPlugin.so"/>
         <contact>
-            <collision>RR_calf_fixed_joint_lump__RR_foot_collision_1</collision>
+            <collision>RH_calf_fixed_joint_lump__RH_foot_collision_1</collision>
         </contact>
         </sensor>
@@ -89,5 +89,5 @@
         <plugin name="contactPlugin" filename="libunitreeFootContactPlugin.so"/>
         <contact>
-            <collision>RL_calf_fixed_joint_lump__RL_foot_collision_1</collision>
+            <collision>LH_calf_fixed_joint_lump__LH_foot_collision_1</collision>
         </contact>
         </sensor>
@@ -97,5 +97,5 @@
         <visual>
             <plugin name="drawForcePlugin" filename="libunitreeDrawForcePlugin.so">
-                <topicName>FR_foot_contact</topicName>
+                <topicName>RF_foot_contact</topicName>
             </plugin>
         </visual>
@@ -104,5 +104,5 @@
         <visual>
             <plugin name="drawForcePlugin" filename="libunitreeDrawForcePlugin.so">
-                <topicName>FL_foot_contact</topicName>
+                <topicName>LF_foot_contact</topicName>
             </plugin>
         </visual>
@@ -111,5 +111,5 @@
         <visual>
             <plugin name="drawForcePlugin" filename="libunitreeDrawForcePlugin.so">
-                <topicName>RR_foot_contact</topicName>
+                <topicName>RH_foot_contact</topicName>
             </plugin>
         </visual>
@@ -118,5 +118,5 @@
         <visual>
             <plugin name="drawForcePlugin" filename="libunitreeDrawForcePlugin.so">
-                <topicName>RL_foot_contact</topicName>
+                <topicName>LH_foot_contact</topicName>
             </plugin>
         </visual>

File: qm_description/urdf/quadruped_manipulator/robot.xacro (robot description, xacro)
@@ -1,4 +1,4 @@
 <?xml version="1.0"?>
-<robot xmlns:xacro="http://www.ros.org/wiki/xacro" name="qm">
+<robot name="qm" xmlns:xacro="http://www.ros.org/wiki/xacro">
     <xacro:arg name="robot_type" default="aliengo"/>
     <xacro:include filename="$(find qm_description)/urdf/quadruped_manipulator/gazebo.xacro"/>
@@ -10,4 +10,5 @@
     <xacro:include filename="$(find qm_description)/urdf/manipulator/const.xacro"/>
     <xacro:include filename="$(find qm_description)/urdf/manipulator/transmission.xacro"/>
+    <xacro:arg name="UnitreeGripper" default="true"/>
     <!-- Debug mode will hung up the robot, use "true" or "false" to switch it. -->
     <xacro:if value="$(arg DEBUG)">
@@ -23,5 +24,18 @@
             <origin rpy="0 0 0" xyz="0 0 0"/>
             <geometry>
-                <mesh filename="package://qm_description/meshes/quadruped/$(arg robot_type)/trunk.dae" scale="1 1 1"/>
+                <box size="0.001 0.001 0.001"/>
+            </geometry>
+        </visual>
+    </link>
+    <joint name="floating_base" type="fixed">
+        <origin rpy="0 0 0" xyz="0 0 0"/>
+        <parent link="base"/>
+        <child link="trunk"/>
+    </joint>
+    <link name="trunk">
+        <visual>
+            <origin rpy="0 0 0" xyz="0 0 0"/>
+            <geometry>
+                 <mesh filename="package://qm_description/meshes/quadruped/$(arg robot_type)/trunk.dae" scale="1 1 1"/>
             </geometry>
         </visual>
@@ -31,4 +45,5 @@
                 <box size="${trunk_length} ${trunk_width} ${trunk_height}"/>
             </geometry>
+            <material name="red"/>
         </collision>
         <inertial>
@@ -36,13 +51,37 @@
             <mass value="${trunk_mass}"/>
             <inertia
-                    ixx="${trunk_ixx}" ixy="${trunk_ixy}" ixz="${trunk_ixz}"
-                    iyy="${trunk_iyy}" iyz="${trunk_iyz}"
-                    izz="${trunk_izz}"/>
-        </inertial>
-    </link>
-     <xacro:IMU connected_to="base" imu_name="unitree_imu" xyz="0. 0. 0." rpy="0. 0. 0."/>
+                ixx="${trunk_ixx}" ixy="${trunk_ixy}" ixz="${trunk_ixz}"
+                iyy="${trunk_iyy}" iyz="${trunk_iyz}"
+                izz="${trunk_izz}"/>
+        </inertial>
+    </link>
+    <joint name="imu_joint" type="fixed">
+        <parent link="trunk"/>
+        <child link="imu_link"/>
+        <origin rpy="0 0 0" xyz="0 0 0"/>
+    </joint>
+    <link name="imu_link">
+        <inertial>
+            <mass value="0.001"/>
+            <origin rpy="0 0 0" xyz="0 0 0"/>
+            <inertia ixx="0.0001" ixy="0" ixz="0" iyy="0.000001" iyz="0" izz="0.0001"/>
+        </inertial>
+        <visual>
+            <origin rpy="0 0 0" xyz="0 0 0"/>
+            <geometry>
+                <box size="0.001 0.001 0.001"/>
+            </geometry>
+            <material name="red"/>
+        </visual>
+        <collision>
+            <origin rpy="0 0 0" xyz="0 0 0"/>
+            <geometry>
+                <box size=".001 .001 .001"/>
+            </geometry>
+        </collision>
+    </link>
     <joint name="trunk_arm_joint" type="fixed">
         <origin rpy="${arm_offset_r} ${arm_offset_p} ${arm_offset_yaw}" xyz="${arm_offset_x} ${arm_offset_y} ${arm_offset_z}"/>
-        <parent link="base"/>
+        <parent link="trunk"/>
         <child link="link00"/>
     </joint>
@@ -82,5 +121,5 @@
             <origin rpy="0 0 0" xyz="0 0 0"/>
             <geometry>
-                <mesh filename="package://qm_description/meshes/manipulator/z1_Link01.stl" scale="1 1 1"/>
+                 <mesh filename="package://qm_description/meshes/manipulator/z1_Link01.stl" scale="1 1 1"/>
             </geometry>
             <material name="silver"/>
@@ -193,5 +232,5 @@
             <origin rpy="0 0 0" xyz="0 0 0"/>
             <geometry>
-                <mesh filename="package://qm_description/meshes/manipulator/z1_Link04.stl" scale="1 1 1"/>
+                 <mesh filename="package://qm_description/meshes/manipulator/z1_Link04.stl" scale="1 1 1"/>
             </geometry>
             <material name="silver"/>
@@ -255,7 +294,7 @@
         <collision>
             <geometry>
-                <cylinder length="${motor_height - 0.01}" radius="${motor_diameter}"/>
-            </geometry>
-            <origin rpy="0 ${PI/2.0} 0" xyz="${(motor_height - 0.01)/2.0} 0 0"/>
+                <cylinder length="${motor_height}" radius="${motor_diameter}"/>
+            </geometry>
+            <origin rpy="0 ${PI/2.0} 0" xyz="${motor_height/2.0} 0 0"/>
         </collision>
         <inertial>
@@ -268,60 +307,70 @@
         </inertial>
     </link>
-    <joint name="gripperStator" type="fixed">
-        <origin rpy="0 0 0" xyz="0.051 0.0 0.0"/>
-        <parent link="link06"/>
-        <child link="gripperStator"/>
-    </joint>
-    <link name="gripperStator">
-        <visual>
-            <geometry>
-                <mesh filename="package://qm_description/meshes/manipulator/z1_GripperStator.stl" scale="1 1 1"/>
-            </geometry>
-            <material name="grey"/>
-        </visual>
-        <collision>
-            <geometry>
-                <mesh filename="package://qm_description/meshes/manipulator/z1_GripperStator.stl" scale="1 1 1"/>
-            </geometry>
-        </collision>
-        <inertial>
-            <origin rpy="0 0 0" xyz="${GripperStator_ComX} ${GripperStator_ComY} ${GripperStator_ComZ}"/>
-            <mass value="${GripperStator_Mass}"/>
-            <inertia
-                ixx="${GripperStator_Ixx}" ixy="${GripperStator_Ixy}" ixz="${GripperStator_Ixz}"
-                iyy="${GripperStator_Iyy}" iyz="${GripperStator_Iyz}"
-                izz="${GripperStator_Izz}"/>
-        </inertial>
-    </link>
-    <joint name="jointGripper" type="revolute">
-        <origin rpy="0 0 0" xyz="0.049 0.0 0"/>
-        <parent link="gripperStator"/>
-        <child link="gripperMover"/>
-        <axis xyz="0 1 0"/>
-        <dynamics damping="${jointDamping}" friction="${jointFriction}"/>
-        <limit effort="${torqueMax}" velocity="${velocityMax}" lower="${Gripper_PositionMin}" upper="${Gripper_PositionMax}"/>
-    </joint>
-    <link name="gripperMover">
-        <visual>
-            <geometry>
-                <mesh filename="package://qm_description/meshes/manipulator/z1_GripperMover.stl" scale="1 1 1"/>
-            </geometry>
-            <material name="grey"/>
-        </visual>
-        <collision>
-            <geometry>
-                <mesh filename="package://qm_description/meshes/manipulator/z1_GripperMover.stl" scale="1 1 1"/>
-            </geometry>
-        </collision>
-        <inertial>
-            <origin rpy="0 0 0" xyz="${GripperMover_ComX} ${GripperMover_ComY} ${GripperMover_ComZ}"/>
-            <mass value="${GripperMover_Mass}"/>
-            <inertia
-                ixx="${GripperMover_Ixx}" ixy="${GripperMover_Ixy}" ixz="${GripperMover_Ixz}"
-                iyy="${GripperMover_Iyy}" iyz="${GripperMover_Iyz}"
-                izz="${GripperMover_Izz}"/>
-        </inertial>
-    </link>
-    <xacro:motorTransmission name="Gripper"/>
+    <xacro:if value="$(arg UnitreeGripper)">
+        <joint name="gripperStator" type="fixed">
+            <origin rpy="0 0 0" xyz="0.051 0.0 0.0"/>
+            <parent link="link06"/>
+            <child link="gripperStator"/>
+        </joint>
+        <link name="gripperStator">
+            <visual>
+                <geometry>
+                    <mesh filename="package://qm_description/meshes/manipulator/z1_GripperStator.stl" scale="1 1 1"/>
+                </geometry>
+                <material name="black"/>
+            </visual>
+            <collision>
+                <geometry>
+                    <mesh filename="package://qm_description/meshes/manipulator/z1_GripperStator.stl" scale="1 1 1"/>
+                </geometry>
+                <material name="green"/>
+            </collision>
+            <inertial>
+                <origin rpy="0 0 0" xyz="${GripperStator_ComX} ${GripperStator_ComY} ${GripperStator_ComZ}"/>
+                <mass value="${GripperStator_Mass}"/>
+                <inertia
+                    ixx="${GripperStator_Ixx}" ixy="${GripperStator_Ixy}" ixz="${GripperStator_Ixz}"
+                    iyy="${GripperStator_Iyy}" iyz="${GripperStator_Iyz}"
+                    izz="${GripperStator_Izz}"/>
+            </inertial>
+        </link>
+        <joint name="jointGripper" type="revolute">
+            <origin rpy="0 0 0" xyz="0.049 0.0 0"/>
+            <parent link="gripperStator"/>
+            <child link="gripperMover"/>
+            <axis xyz="0 1 0"/>
+            <dynamics damping="${jointDamping}" friction="${jointFriction}"/>
+            <limit effort="${torqueMax}" velocity="${velocityMax}" lower="${Gripper_PositionMin}" upper="${Gripper_PositionMax}"/>
+        </joint>
+        <link name="gripperMover">
+            <visual>
+                <geometry>
+                    <mesh filename="package://qm_description/meshes/manipulator/z1_GripperMover.stl" scale="1 1 1"/>
+                </geometry>
+                <material name="black"/>
+            </visual>
+            <collision>
+                <geometry>
+                    <mesh filename="package://qm_description/meshes/manipulator/z1_GripperMover.stl" scale="1 1 1"/>
+                </geometry>
+                <material name="green"/>
+            </collision>
+            <inertial>
+                <origin rpy="0 0 0" xyz="${GripperMover_ComX} ${GripperMover_ComY} ${GripperMover_ComZ}"/>
+                <mass value="${GripperMover_Mass}"/>
+                <inertia
+                    ixx="${GripperMover_Ixx}" ixy="${GripperMover_Ixy}" ixz="${GripperMover_Ixz}"
+                    iyy="${GripperMover_Iyy}" iyz="${GripperMover_Iyz}"
+                    izz="${GripperMover_Izz}"/>
+            </inertial>
+        </link>
+        <xacro:motorTransmission name="Gripper"/>
+        <gazebo reference="gripperStator">
+            <self_collide>true</self_collide>
+        </gazebo>
+        <gazebo reference="gripperMover">
+            <self_collide>true</self_collide>
+        </gazebo>
+    </xacro:if>
     <xacro:motorTransmission name="1"/>
     <xacro:motorTransmission name="2"/>
