Commit message: Updates vision and planning packages

File: qm_description/urdf/quadruped_manipulator/camera.xacro (robot description, xacro)
@@ -47,5 +47,5 @@
                 <pointCloudTopicName>depth/color/points</pointCloudTopicName>
                 <frameName>camera_link_optical</frameName>
-                <pointCloudCutoff>0.2</pointCloudCutoff>
+                <pointCloudCutoff>0.02</pointCloudCutoff>
                 <pointCloudCutoffMax>4.0</pointCloudCutoffMax>
             </plugin>

File: qm_description/urdf/quadruped_manipulator/robot.xacro (robot description, xacro)
@@ -520,4 +520,18 @@
                 <material name="red"/>
             </visual>
+            <inertial>
+                <mass value="0.0"/>
+                <inertia ixx="0.0" ixy="0.0" ixz="0.0" iyy="0.0" iyz="0.0" izz="0.0"/>
+            </inertial>
+            <collision>
+                <geometry>
+                    <sphere radius="0.01"/>
+                </geometry>
+                <surface>
+                    <contact>
+                        <collide_bitmask>0</collide_bitmask>
+                    </contact>
+                </surface>
+            </collision>
         </link>
         <joint name="z1_joint_end_effector" type="fixed">
