Commit message: Update vision module

File: qm_description/urdf/quadruped_manipulator/const.xacro (robot description, xacro)
@@ -2,8 +2,9 @@
 <robot name="aliengoZ1_description" xmlns:xacro="http://www.ros.org/wiki/xacro">
     <xacro:include filename="$(find qm_description)/urdf/quadruped/aliengo/const.xacro"/>
+<!-- - 0.145  + 0.02-->
       <!-- the base of arm offset -->
     <xacro:property name="arm_offset_x" value="${trunk_length/2.0 - 0.07}"/>
     <xacro:property name="arm_offset_y" value="0"/>
-    <xacro:property name="arm_offset_z" value="${trunk_height/2.0}"/>
+    <xacro:property name="arm_offset_z" value="${trunk_height/2.0 }"/>
     <xacro:property name="arm_offset_r" value="0"/>
     <xacro:property name="arm_offset_p" value="0"/>

File: qm_description/urdf/quadruped_manipulator/robot.xacro (robot description, xacro)
@@ -490,5 +490,19 @@
             <limit effort="${torqueMax}" velocity="${velocityMax}" lower="${Gripper_PositionMin}" upper="${Gripper_PositionMax}"/>
         </joint>
-        <xacro:motorTransmission name="Gripper"/>
+        <transmission name="z1_joint_Gripper_trans">
+            <type>transmission_interface/SimpleTransmission</type>
+            <joint name="z1_joint_Gripper">
+                <hardwareInterface>hardware_interface/EffortJointInterface</hardwareInterface>
+            </joint>
+            <actuator name="z1_joint_Gripper_motor">
+                <mechanicalReduction>1</mechanicalReduction>
+            </actuator>
+        </transmission>
+        <!-- <gazebo>
+            <plugin name="gripper_position_controller" filename="libgazebo_ros_control_select_joints.so">
+                <robotNamespace>/</robotNamespace>
+                <joints>z1_joint_Gripper</joints>
+            </plugin>
+        </gazebo> -->
         <link name="gripperMover">
             <visual>
