Commit message: :bug: BUG: Update .dae path

File: qm_description/urdf/quadruped_manipulator/camera2.xacro (robot description, xacro)
@@ -44,5 +44,5 @@
             <origin xyz="${d435_zero_depth_to_glass + d435_glass_to_front} ${-d435_cam_depth_py} 0" rpy="${M_PI/2} 0 ${M_PI/2}"/>
             <geometry>
-                <mesh filename="file://$(find realsense2_description)/meshes/d435.dae" />
+                <mesh filename="file://$(find qm_description)/meshes/camera/d435.dae" />
             </geometry>
             <material name="black">  <!-- Add the name attribute here -->
