Commit message: Controller correction

File: qm_description/urdf/manipulator/transmission.xacro (robot description, xacro)
@@ -2,10 +2,10 @@
 <robot xmlns:xacro="http://www.ros.org/wiki/xacro">
     <xacro:macro name="motorTransmission" params="name">
-        <transmission name="JointTrans${name}">
+        <transmission name="z1_joint_${name}_trans">
             <type>transmission_interface/SimpleTransmission</type>
             <joint name="joint${name}">
                 <hardwareInterface>hardware_interface/EffortJointInterface</hardwareInterface>
             </joint>
-            <actuator name="Actuator${name}">
+            <actuator name="z1_joint_${name}_actuator">
                 <hardwareInterface>hardware_interface/EffortJointInterface</hardwareInterface>
                 <mechanicalReduction>1</mechanicalReduction>

File: qm_description/urdf/quadruped_manipulator/gazebo.xacro (robot description, xacro)
@@ -1,12 +1,4 @@
 <?xml version="1.0"?>
 <robot>
-    <!-- ros_control plugin -->
-    <!-- <gazebo>
-        <plugin name="gazebo_ros_control" filename="liblegged_hw_sim.so">
-            <robotNamespace>/</robotNamespace>
-            <robotParam>legged_robot_description</robotParam>
-            <robotSimType>legged_gazebo/LeggedHWSim</robotSimType>
-        </plugin>
-    </gazebo> -->
     <gazebo>
         <plugin name="p3d_base_controller" filename="libgazebo_ros_p3d.so">
@@ -35,5 +27,5 @@
         <mu1>0.2</mu1>
         <mu2>0.2</mu2>
-        <material>Gazebo/DarkGrey</material>
+        <material>Gazebo/Black</material>
     </gazebo>
     <gazebo reference="LF_thigh">
@@ -41,5 +33,5 @@
         <mu2>0.2</mu2>
         <self_collide>0</self_collide>
-        <material>Gazebo/DarkGrey</material>
+        <material>Gazebo/Black</material>
         <kp value="1000000.0"/>
         <kd value="1.0"/>
@@ -49,4 +41,5 @@
         <mu2>0.2</mu2>
         <self_collide>1</self_collide>
+        <material>Gazebo/Black</material>
     </gazebo>
     <gazebo reference="LF_FOOT">
@@ -54,5 +47,5 @@
         <mu2>0.6</mu2>
         <self_collide>1</self_collide>
-        <material>Gazebo/DarkGrey</material>
+        <material>Gazebo/Black</material>
         <kp value="1000000.0"/>
         <kd value="1.0"/>
@@ -62,5 +55,5 @@
         <mu1>0.2</mu1>
         <mu2>0.2</mu2>
-        <material>Gazebo/DarkGrey</material>
+        <material>Gazebo/Black</material>
     </gazebo>
     <gazebo reference="RF_thigh">
@@ -68,5 +61,5 @@
         <mu2>0.2</mu2>
         <self_collide>0</self_collide>
-        <material>Gazebo/DarkGrey</material>
+        <material>Gazebo/Black</material>
         <kp value="1000000.0"/>
         <kd value="1.0"/>
@@ -76,4 +69,5 @@
         <mu2>0.2</mu2>
         <self_collide>1</self_collide>
+        <material>Gazebo/Black</material>
     </gazebo>
     <gazebo reference="RF_FOOT">
@@ -81,5 +75,5 @@
         <mu2>0.6</mu2>
         <self_collide>1</self_collide>
-        <material>Gazebo/DarkGrey</material>
+        <material>Gazebo/Black</material>
         <kp value="1000000.0"/>
         <kd value="1.0"/>
@@ -89,5 +83,5 @@
         <mu1>0.2</mu1>
         <mu2>0.2</mu2>
-        <material>Gazebo/DarkGrey</material>
+        <material>Gazebo/Black</material>
     </gazebo>
     <gazebo reference="LH_thigh">
@@ -95,5 +89,5 @@
         <mu2>0.2</mu2>
         <self_collide>0</self_collide>
-        <material>Gazebo/DarkGrey</material>
+        <material>Gazebo/Black</material>
         <kp value="1000000.0"/>
         <kd value="1.0"/>
@@ -103,4 +97,5 @@
         <mu2>0.2</mu2>
         <self_collide>1</self_collide>
+        <material>Gazebo/Black</material>
     </gazebo>
     <gazebo reference="LH_FOOT">
@@ -108,5 +103,5 @@
         <mu2>0.6</mu2>
         <self_collide>1</self_collide>
-        <material>Gazebo/DarkGrey</material>
+        <material>Gazebo/Black</material>
         <kp value="1000000.0"/>
         <kd value="1.0"/>
@@ -116,5 +111,5 @@
         <mu1>0.2</mu1>
         <mu2>0.2</mu2>
-        <material>Gazebo/DarkGrey</material>
+        <material>Gazebo/Black</material>
     </gazebo>
     <gazebo reference="RH_thigh">
@@ -122,5 +117,5 @@
         <mu2>0.2</mu2>
         <self_collide>0</self_collide>
-        <material>Gazebo/DarkGrey</material>
+        <material>Gazebo/Black</material>
         <kp value="1000000.0"/>
         <kd value="1.0"/>
@@ -130,4 +125,5 @@
         <mu2>0.2</mu2>
         <self_collide>1</self_collide>
+        <material>Gazebo/Black</material>
     </gazebo>
     <gazebo reference="RH_FOOT">
@@ -135,7 +131,46 @@
         <mu2>0.6</mu2>
         <self_collide>1</self_collide>
-        <material>Gazebo/DarkGrey</material>
+        <material>Gazebo/Black</material>
         <kp value="1000000.0"/>
         <kd value="1.0"/>
     </gazebo>
+    <!-- Z1 arm -->
+     <gazebo reference="link00">
+        <material>Gazebo/Grey</material>
+    </gazebo>
+     <gazebo reference="link01">
+        <material>Gazebo/Grey</material>
+        <provideFeedback>true</provideFeedback>
+    </gazebo>
+    <gazebo reference="link02">
+        <material>Gazebo/Grey</material>
+        <provideFeedback>true</provideFeedback>
+    </gazebo>
+    <gazebo reference="link03">
+        <material>Gazebo/Grey</material>
+        <provideFeedback>true</provideFeedback>
+    </gazebo>
+    <gazebo reference="link04">
+        <self_collide>true</self_collide>
+        <material>Gazebo/Grey</material>
+        <provideFeedback>true</provideFeedback>
+    </gazebo>
+    <gazebo reference="link05">
+        <self_collide>true</self_collide>
+        <material>Gazebo/Grey</material>
+        <provideFeedback>true</provideFeedback>
+    </gazebo>
+    <gazebo reference="link06">
+        <self_collide>true</self_collide>
+        <material>Gazebo/Grey</material>
+        <provideFeedback>true</provideFeedback>
+    </gazebo>
+    <gazebo reference="gripperStator">
+        <self_collide>true</self_collide>
+        <material>Gazebo/Black</material>
+    </gazebo>
+    <gazebo reference="gripperMover">
+        <self_collide>true</self_collide>
+        <material>Gazebo/Black</material>
+    </gazebo>
 </robot>

File: qm_description/urdf/quadruped_manipulator/robot.urdf (robot description, URDF)
Before this commit: robot qm, 28 links, 27 joints
Links:
- removed link imu_link
- removed link trunk
- added link unitree_imu, mass 0.01; visual box size=0.015 0.015 0.004
- added link z1_end_effector; visual sphere radius=0.01
- link base: mass None -> 11.041; geometry collision box size=0.647 0.15 0.112; visual mesh filename=package://qm_description/meshes/quadruped/aliengo/trunk.dae scale=1 1 1
Joints:
- removed joint floating_base
- removed joint imu_joint
- removed joint trunk_arm_joint
- added joint manipulator_joint: type fixed, parent base, child link00, origin xyz=0.2535 0 0.056 rpy=0 0 0
- added joint unitree_imu_joint: type fixed, parent base, child unitree_imu, origin xyz=0. 0. 0. rpy=0. 0. 0.
- added joint z1_joint_end_effector: type fixed, parent gripperStator, child z1_end_effector, origin xyz=0.135 0 0 rpy=0 0 0

File: qm_description/urdf/quadruped_manipulator/robot.xacro (robot description, xacro)
@@ -4,5 +4,5 @@
     <xacro:include filename="$(find qm_description)/urdf/quadruped/common/materials.xacro"/>
     <xacro:include filename="$(find qm_description)/urdf/quadruped/common/leg.xacro"/>
-    <xacro:include filename="$(find qm_description)/urdf/quadruped_manipulator/gazebo_original.xacro"/>
+    <xacro:include filename="$(find qm_description)/urdf/quadruped_manipulator/gazebo.xacro"/>
     <xacro:include filename="$(find qm_description)/urdf/quadruped/common/imu.xacro"/>
     <xacro:include filename="$(find qm_description)/urdf/quadruped/aliengo/const.xacro"/>
@@ -11,31 +11,10 @@
     <xacro:include filename="$(find qm_description)/urdf/manipulator/transmission.xacro"/>
     <xacro:arg name="UnitreeGripper" default="true"/>
-    <!-- Debug mode will hung up the robot, use "true" or "false" to switch it. -->
-    <xacro:if value="$(arg DEBUG)">
-        <link name="world"/>
-        <joint name="base_static_joint" type="fixed">
-            <origin rpy="0 0 0" xyz="0 0 0"/>
-            <parent link="world"/>
-            <child link="base"/>
-        </joint>
-    </xacro:if>
-    <link name="base">
-        <visual>
-            <origin rpy="0 0 0" xyz="0 0 0"/>
-            <geometry>
-                <box size="0.001 0.001 0.001"/>
-            </geometry>
-        </visual>
-    </link>
-    <joint name="floating_base" type="fixed">
-        <origin rpy="0 0 0" xyz="0 0 0"/>
-        <parent link="base"/>
-        <child link="trunk"/>
-    </joint>
-    <link name="trunk">
-        <visual>
-            <origin rpy="0 0 0" xyz="0 0 0"/>
-            <geometry>
-                 <mesh filename="package://qm_description/meshes/quadruped/$(arg robot_type)/trunk.dae" scale="1 1 1"/>
+     <!-- Aliengo robot -->
+     <link name="base">
+        <visual>
+            <origin rpy="0 0 0" xyz="0 0 0"/>
+            <geometry>
+                <mesh filename="package://qm_description/meshes/quadruped/$(arg robot_type)/trunk.dae" scale="1 1 1"/>
             </geometry>
         </visual>
@@ -45,5 +24,4 @@
                 <box size="${trunk_length} ${trunk_width} ${trunk_height}"/>
             </geometry>
-            <material name="red"/>
         </collision>
         <inertial>
@@ -51,40 +29,31 @@
             <mass value="${trunk_mass}"/>
             <inertia
-                ixx="${trunk_ixx}" ixy="${trunk_ixy}" ixz="${trunk_ixz}"
-                iyy="${trunk_iyy}" iyz="${trunk_iyz}"
-                izz="${trunk_izz}"/>
-        </inertial>
-    </link>
-    <joint name="imu_joint" type="fixed">
-        <parent link="trunk"/>
-        <child link="imu_link"/>
-        <origin rpy="0 0 0" xyz="0 0 0"/>
-    </joint>
-    <link name="imu_link">
-        <inertial>
-            <mass value="0.001"/>
-            <origin rpy="0 0 0" xyz="0 0 0"/>
-            <inertia ixx="0.0001" ixy="0" ixz="0" iyy="0.000001" iyz="0" izz="0.0001"/>
-        </inertial>
-        <visual>
-            <origin rpy="0 0 0" xyz="0 0 0"/>
-            <geometry>
-                <box size="0.001 0.001 0.001"/>
-            </geometry>
-            <material name="red"/>
-        </visual>
-        <collision>
-            <origin rpy="0 0 0" xyz="0 0 0"/>
-            <geometry>
-                <box size=".001 .001 .001"/>
-            </geometry>
-        </collision>
-    </link>
-    <joint name="trunk_arm_joint" type="fixed">
+                    ixx="${trunk_ixx}" ixy="${trunk_ixy}" ixz="${trunk_ixz}"
+                    iyy="${trunk_iyy}" iyz="${trunk_iyz}"
+                    izz="${trunk_izz}"/>
+        </inertial>
+    </link>
+    <!-- IMU -->
+    <xacro:IMU connected_to="base" imu_name="unitree_imu" xyz="0. 0. 0." rpy="0. 0. 0."/>
+    <!-- Aliengo legs -->
+    <xacro:leg prefix="RF" mirror="-1" mirror_dae="False" front_hind="1" front_hind_dae="True">
+        <origin rpy="0 0 0" xyz="${leg_offset_x} ${-leg_offset_y} 0"/>
+    </xacro:leg>
+    <xacro:leg prefix="LF" mirror="1" mirror_dae="True" front_hind="1" front_hind_dae="True">
+        <origin rpy="0 0 0" xyz="${leg_offset_x} ${leg_offset_y} 0"/>
+    </xacro:leg>
+    <xacro:leg prefix="RH" mirror="-1" mirror_dae="False" front_hind="-1" front_hind_dae="False">
+        <origin rpy="0 0 0" xyz="${-leg_offset_x} ${-leg_offset_y} 0"/>
+    </xacro:leg>
+    <xacro:leg prefix="LH" mirror="1" mirror_dae="True" front_hind="-1" front_hind_dae="False">
+        <origin rpy="0 0 0" xyz="${-leg_offset_x} ${leg_offset_y} 0"/>
+    </xacro:leg>
+    <!-- Z1 manipulator -->
+    <joint name="manipulator_joint" type="fixed">
         <origin rpy="${arm_offset_r} ${arm_offset_p} ${arm_offset_yaw}" xyz="${arm_offset_x} ${arm_offset_y} ${arm_offset_z}"/>
-        <parent link="trunk"/>
+        <parent link="base"/>
         <child link="link00"/>
     </joint>
-     <link name="link00">
+    <link name="link00">
         <visual>
             <origin rpy="0 0 0" xyz="0 0 0"/>
@@ -117,4 +86,12 @@
         <limit effort="${torqueMax}" velocity="${velocityMax}" lower="${joint1_PositionMin}" upper="${joint1_PositionMax}"/>
     </joint>
+    <xacro:motorTransmission name="1"/>
+    <gazebo>
+        <plugin filename="libgazebo_ros_ft_sensor.so" name="ft_sensor">
+        <updateRate>30.0</updateRate>
+        <topicName>joint1_ft_sensor_topic</topicName>
+        <jointName>joint1</jointName>
+        </plugin>
+    </gazebo>
     <link name="link01">
         <visual>
@@ -148,4 +125,12 @@
         <limit effort="${2*torqueMax}" velocity="${velocityMax}" lower="${joint2_PositionMin}" upper="${joint2_PositionMax}"/>
     </joint>
+    <xacro:motorTransmission name="2"/>
+    <gazebo>
+        <plugin filename="libgazebo_ros_ft_sensor.so" name="ft_sensor">
+        <updateRate>30.0</updateRate>
+        <topicName>joint2_ft_sensor_topic</topicName>
+        <jointName>joint2</jointName>
+        </plugin>
+    </gazebo>
     <link name="link02">
         <visual>
@@ -191,4 +176,12 @@
         <limit effort="${torqueMax}" velocity="${velocityMax}" lower="${joint3_PositionMin}" upper="${joint3_PositionMax}"/>
     </joint>
+    <xacro:motorTransmission name="3"/>
+    <gazebo>
+        <plugin filename="libgazebo_ros_ft_sensor.so" name="ft_sensor">
+        <updateRate>30.0</updateRate>
+        <topicName>joint3_ft_sensor_topic</topicName>
+        <jointName>joint3</jointName>
+        </plugin>
+    </gazebo>
     <link name="link03">
         <visual>
@@ -228,4 +221,12 @@
         <limit effort="${torqueMax}" velocity="${velocityMax}" lower="${joint4_PositionMin}" upper="${joint4_PositionMax}"/>
     </joint>
+    <xacro:motorTransmission name="4"/>
+    <gazebo>
+        <plugin filename="libgazebo_ros_ft_sensor.so" name="ft_sensor">
+        <updateRate>30.0</updateRate>
+        <topicName>joint4_ft_sensor_topic</topicName>
+        <jointName>joint4</jointName>
+        </plugin>
+    </gazebo>
     <link name="link04">
         <visual>
@@ -259,4 +260,12 @@
         <limit effort="${torqueMax}" velocity="${velocityMax}" lower="${joint5_PositionMin}" upper="${joint5_PositionMax}"/>
     </joint>
+    <xacro:motorTransmission name="5"/>
+    <gazebo>
+        <plugin filename="libgazebo_ros_ft_sensor.so" name="ft_sensor">
+        <updateRate>30.0</updateRate>
+        <topicName>joint5_ft_sensor_topic</topicName>
+        <jointName>joint5</jointName>
+        </plugin>
+    </gazebo>
     <link name="link05">
         <visual>
@@ -284,4 +293,12 @@
         <limit effort="${torqueMax}" velocity="${velocityMax}" lower="${joint6_PositionMin}" upper="${joint6_PositionMax}"/>
     </joint>
+    <xacro:motorTransmission name="6"/>
+    <gazebo>
+        <plugin filename="libgazebo_ros_ft_sensor.so" name="ft_sensor">
+        <updateRate>30.0</updateRate>
+        <topicName>joint6_ft_sensor_topic</topicName>
+        <jointName>joint6</jointName>
+        </plugin>
+    </gazebo>
     <link name="link06">
         <visual>
@@ -335,17 +352,4 @@
             </inertial>
         </link>
-        <link name="z1_end_effector">
-            <visual>
-                <geometry>
-                    <sphere radius="0.01"/>
-                </geometry>
-                <material name="red"/>
-            </visual>
-        </link>
-        <joint name="z1_joint_end_effector" type="fixed">
-            <origin xyz="0.135 0 0" rpy="0 0 0"/>
-            <parent link="gripperStator"/>
-            <child link="z1_end_effector"/>
-        </joint>
         <joint name="jointGripper" type="revolute">
             <origin rpy="0 0 0" xyz="0.049 0.0 0"/>
@@ -379,29 +383,18 @@
         </link>
         <xacro:motorTransmission name="Gripper"/>
-        <gazebo reference="gripperStator">
-            <self_collide>true</self_collide>
-        </gazebo>
-        <gazebo reference="gripperMover">
-            <self_collide>true</self_collide>
-        </gazebo>
+        <link name="z1_end_effector">
+            <visual>
+                <geometry>
+                    <sphere radius="0.01"/>
+                </geometry>
+                <material name="red"/>
+            </visual>
+        </link>
+        <joint name="z1_joint_end_effector" type="fixed">
+            <origin xyz="0.135 0 0" rpy="0 0 0"/>
+            <parent link="gripperStator"/>
+            <child link="z1_end_effector"/>
+        </joint>
     </xacro:if>
-    <xacro:motorTransmission name="1"/>
-    <xacro:motorTransmission name="2"/>
-    <xacro:motorTransmission name="3"/>
-    <xacro:motorTransmission name="4"/>
-    <xacro:motorTransmission name="5"/>
-    <xacro:motorTransmission name="6"/>
-    <xacro:leg prefix="RF" mirror="-1" mirror_dae="False" front_hind="1" front_hind_dae="True">
-        <origin rpy="0 0 0" xyz="${leg_offset_x} ${-leg_offset_y} 0"/>
-    </xacro:leg>
-    <xacro:leg prefix="LF" mirror="1" mirror_dae="True" front_hind="1" front_hind_dae="True">
-        <origin rpy="0 0 0" xyz="${leg_offset_x} ${leg_offset_y} 0"/>
-    </xacro:leg>
-    <xacro:leg prefix="RH" mirror="-1" mirror_dae="False" front_hind="-1" front_hind_dae="False">
-        <origin rpy="0 0 0" xyz="${-leg_offset_x} ${-leg_offset_y} 0"/>
-    </xacro:leg>
-    <xacro:leg prefix="LH" mirror="1" mirror_dae="True" front_hind="-1" front_hind_dae="False">
-        <origin rpy="0 0 0" xyz="${-leg_offset_x} ${leg_offset_y} 0"/>
-    </xacro:leg>
     <!-- ros_control plugin -->
     <gazebo>
