Commit message: Z1 qm URDF

File: qm_description/urdf/manipulator/gazebo.xacro (robot description, xacro)
@@ -9,10 +9,13 @@
     <gazebo reference="link04">
         <self_collide>true</self_collide>
+        <material>Gazebo/DarkGrey</material>
     </gazebo>
     <gazebo reference="link05">
         <self_collide>true</self_collide>
+        <material>Gazebo/DarkGrey</material>
     </gazebo>
     <gazebo reference="link06">
         <self_collide>true</self_collide>
+        <material>Gazebo/DarkGrey</material>
     </gazebo>
 </robot>

File: qm_description/urdf/manipulator/robot.xacro (robot description, xacro)
@@ -1,14 +1,9 @@
 <?xml version="1.0"?>
-<robot name="z1" xmlns:xacro="http://www.ros.org/wiki/xacro">
-    <xacro:include filename="$(find qm_description)/urdf/manipulator/const.xacro"/>
+<robot xmlns:xacro="http://www.ros.org/wiki/xacro" name="robot">
+    <xacro:include filename="$(find qm_description)/urdf/manipulator/materials.xacro"/>
     <xacro:include filename="$(find qm_description)/urdf/manipulator/gazebo.xacro"/>
     <xacro:include filename="$(find qm_description)/urdf/manipulator/transmission.xacro"/>
-    <xacro:arg name="UnitreeGripper" default="true"/>
-    <material name="black">
-        <color rgba="0.0 0.0 0.0 1.0"/>
-    </material>
-    <material name="silver">
-        <color rgba="0.9137254901960784 0.9137254901960784 0.8470588235294118 1.0"/>
-    </material>
+    <xacro:include filename="$(find qm_description)/urdf/manipulator/const.xacro"/>
+    <xacro:arg name="UnitreeGripper" default="false"/>
     <link name="world"/>
     <joint name="base_static_joint" type="fixed">
@@ -21,5 +16,5 @@
             <origin rpy="0 0 0" xyz="0 0 0"/>
             <geometry>
-                <mesh filename="package://qm_description/meshes/manipulator/z1_Link00.dae" scale="1 1 1"/>
+                <mesh filename="package://qm_description/meshes/manipulator/z1_Link00.stl" scale="1 1 1"/>
             </geometry>
             <material name="silver"/>
@@ -52,5 +47,5 @@
             <origin rpy="0 0 0" xyz="0 0 0"/>
             <geometry>
-                <mesh filename="package://qm_description/meshes/manipulator/z1_Link01.dae" scale="1 1 1"/>
+                <mesh filename="package://qm_description/meshes/manipulator/z1_Link01.stl" scale="1 1 1"/>
             </geometry>
             <material name="silver"/>
@@ -77,5 +72,5 @@
             <origin rpy="0 0 0" xyz="0 0 0"/>
             <geometry>
-                <mesh filename="package://qm_description/meshes/manipulator/z1_Link02.dae" scale="1 1 1"/>
+                <mesh filename="package://qm_description/meshes/manipulator/z1_Link02.stl" scale="1 1 1"/>
             </geometry>
             <material name="silver"/>
@@ -120,5 +115,5 @@
             <origin rpy="0 0 0" xyz="0 0 0"/>
             <geometry>
-                <mesh filename="package://qm_description/meshes/manipulator/z1_Link03.dae" scale="1 1 1"/>
+                <mesh filename="package://qm_description/meshes/manipulator/z1_Link03.stl" scale="1 1 1"/>
             </geometry>
             <material name="silver"/>
@@ -157,5 +152,5 @@
             <origin rpy="0 0 0" xyz="0 0 0"/>
             <geometry>
-                <mesh filename="package://qm_description/meshes/manipulator/z1_Link04.dae" scale="1 1 1"/>
+                <mesh filename="package://qm_description/meshes/manipulator/z1_Link04.stl" scale="1 1 1"/>
             </geometry>
             <material name="silver"/>
@@ -188,5 +183,5 @@
             <origin rpy="0 0 0" xyz="0 0 0"/>
             <geometry>
-                <mesh filename="package://qm_description/meshes/manipulator/z1_Link05.dae" scale="1 1 1"/>
+                <mesh filename="package://qm_description/meshes/manipulator/z1_Link05.stl" scale="1 1 1"/>
             </geometry>
             <material name="silver"/>
@@ -213,5 +208,5 @@
             <origin rpy="0 0 0" xyz="0 0 0"/>
             <geometry>
-                <mesh filename="package://qm_description/meshes/manipulator/z1_Link06.dae" scale="1 1 1"/>
+                <mesh filename="package://qm_description/meshes/manipulator/z1_Link06.stl" scale="1 1 1"/>
             </geometry>
             <material name="silver"/>
@@ -241,7 +236,7 @@
             <visual>
                 <geometry>
-                    <mesh filename="package://qm_description/meshes/manipulator/z1_GripperStator.dae" scale="1 1 1"/>
-                </geometry>
-                <material name="black"/>
+                    <mesh filename="package://qm_description/meshes/manipulator/z1_GripperStator.stl" scale="1 1 1"/>
+                </geometry>
+                <material name="grey"/>
             </visual>
             <collision>
@@ -270,7 +265,7 @@
             <visual>
                 <geometry>
-                    <mesh filename="package://qm_description/meshes/manipulator/z1_GripperMover.dae" scale="1 1 1"/>
-                </geometry>
-                <material name="black"/>
+                    <mesh filename="package://qm_description/meshes/manipulator/z1_GripperMover.stl" scale="1 1 1"/>
+                </geometry>
+                <material name="grey"/>
             </visual>
             <collision>

File: qm_description/urdf/manipulator/z1.urdf (robot description, URDF)
Before this commit: robot z1, 8 links, 7 joints
Links:
- link link00: geometry collision cylinder length=0.051 radius=0.0325; visual mesh filename=package://qm_description/meshes/manipulator/z1_Link00.stl scale=1 1 1
- link link01: geometry visual mesh filename=package://qm_description/meshes/manipulator/z1_Link01.stl scale=1 1 1
- link link02: geometry collision cylinder length=0.051 radius=0.0325; collision cylinder length=0.102 radius=0.0325
- link link03: geometry collision cylinder length=0.059 radius=0.0325; collision cylinder length=0.116 radius=0.02
- link link04: geometry collision cylinder length=0.067 radius=0.0325; visual mesh filename=package://qm_description/meshes/manipulator/z1_Link04.stl scale=1 1 1
- link link05: geometry visual mesh filename=package://qm_description/meshes/manipulator/z1_Link05.stl scale=1 1 1
- link link06: geometry collision cylinder length=0.051 radius=0.0325; visual mesh filename=package://qm_description/meshes/manipulator/z1_Link06.stl scale=1 1 1

File: qm_description/urdf/quadruped/aliengo/const.xacro (robot description, xacro)
@@ -36,6 +36,6 @@
     <xacro:property name="hip_velocity_max" value="20"/>
     <xacro:property name="hip_torque_max" value="35.278"/>
-    <xacro:property name="thigh_max" value="1e22"/>
-    <xacro:property name="thigh_min" value="-1e22"/>
+    <xacro:property name="thigh_max" value="${240*pi/180.0}"/>     <!-- 1e22 -->
+    <xacro:property name="thigh_min" value="${-120*pi/180.0}"/>    <!-- -1e22 -->
     <xacro:property name="thigh_velocity_max" value="20"/>
     <xacro:property name="thigh_torque_max" value="35.278"/>

File: qm_description/urdf/quadruped/common/gazebo.xacro (robot description, xacro)
@@ -35,5 +35,5 @@
         <mu1>0.2</mu1>
         <mu2>0.2</mu2>
-        <material>Gazebo/DarkGrey</material>
+        <material>Gazebo/Black</material>
     </gazebo>
     <gazebo reference="LF_thigh">
@@ -41,5 +41,5 @@
         <mu2>0.2</mu2>
         <self_collide>0</self_collide>
-        <material>Gazebo/DarkGrey</material>
+        <material>Gazebo/Black</material>
         <kp value="1000000.0"/>
         <kd value="1.0"/>
@@ -49,4 +49,5 @@
         <mu2>0.2</mu2>
         <self_collide>1</self_collide>
+        <material>Gazebo/Black</material>
     </gazebo>
     <gazebo reference="LF_FOOT">
@@ -54,5 +55,5 @@
         <mu2>0.6</mu2>
         <self_collide>1</self_collide>
-        <material>Gazebo/DarkGrey</material>
+        <material>Gazebo/Black</material>
         <kp value="1000000.0"/>
         <kd value="1.0"/>
@@ -62,5 +63,5 @@
         <mu1>0.2</mu1>
         <mu2>0.2</mu2>
-        <material>Gazebo/DarkGrey</material>
+        <material>Gazebo/Black</material>
     </gazebo>
     <gazebo reference="RF_thigh">
@@ -68,5 +69,5 @@
         <mu2>0.2</mu2>
         <self_collide>0</self_collide>
-        <material>Gazebo/DarkGrey</material>
+        <material>Gazebo/Black</material>
         <kp value="1000000.0"/>
         <kd value="1.0"/>
@@ -76,4 +77,5 @@
         <mu2>0.2</mu2>
         <self_collide>1</self_collide>
+        <material>Gazebo/Black</material>
     </gazebo>
     <gazebo reference="RF_FOOT">
@@ -81,5 +83,5 @@
         <mu2>0.6</mu2>
         <self_collide>1</self_collide>
-        <material>Gazebo/DarkGrey</material>
+        <material>Gazebo/Black</material>
         <kp value="1000000.0"/>
         <kd value="1.0"/>
@@ -89,5 +91,5 @@
         <mu1>0.2</mu1>
         <mu2>0.2</mu2>
-        <material>Gazebo/DarkGrey</material>
+        <material>Gazebo/Black</material>
     </gazebo>
     <gazebo reference="LH_thigh">
@@ -95,5 +97,5 @@
         <mu2>0.2</mu2>
         <self_collide>0</self_collide>
-        <material>Gazebo/DarkGrey</material>
+        <material>Gazebo/Black</material>
         <kp value="1000000.0"/>
         <kd value="1.0"/>
@@ -103,4 +105,5 @@
         <mu2>0.2</mu2>
         <self_collide>1</self_collide>
+        <material>Gazebo/Black</material>
     </gazebo>
     <gazebo reference="LH_FOOT">
@@ -108,5 +111,5 @@
         <mu2>0.6</mu2>
         <self_collide>1</self_collide>
-        <material>Gazebo/DarkGrey</material>
+        <material>Gazebo/Black</material>
         <kp value="1000000.0"/>
         <kd value="1.0"/>
@@ -116,5 +119,5 @@
         <mu1>0.2</mu1>
         <mu2>0.2</mu2>
-        <material>Gazebo/DarkGrey</material>
+        <material>Gazebo/Black</material>
     </gazebo>
     <gazebo reference="RH_thigh">
@@ -122,5 +125,5 @@
         <mu2>0.2</mu2>
         <self_collide>0</self_collide>
-        <material>Gazebo/DarkGrey</material>
+        <material>Gazebo/Black</material>
         <kp value="1000000.0"/>
         <kd value="1.0"/>
@@ -130,4 +133,5 @@
         <mu2>0.2</mu2>
         <self_collide>1</self_collide>
+        <material>Gazebo/Black</material>
     </gazebo>
     <gazebo reference="RH_FOOT">
@@ -135,5 +139,5 @@
         <mu2>0.6</mu2>
         <self_collide>1</self_collide>
-        <material>Gazebo/DarkGrey</material>
+        <material>Gazebo/Black</material>
         <kp value="1000000.0"/>
         <kd value="1.0"/>

File: qm_description/urdf/quadruped/common/materials.xacro (robot description, xacro)
@@ -14,5 +14,5 @@
     </material>
     <material name="silver">
-        <color rgba="${233/255} ${233/255} ${216/255} 1.0"/>
+        <color rgba="${199/255} ${204/255} ${214/255} 1.0"/>
     </material>
     <material name="orange">

File: qm_description/urdf/quadruped_manipulator/robot.urdf (robot description, URDF)
Before this commit: robot qm, 27 links, 26 joints
Links:
- removed link arm_base_link
- removed link j2n6s300_end_effector
- removed link j2n6s300_link_1
- removed link j2n6s300_link_2
- removed link j2n6s300_link_3
- removed link j2n6s300_link_4
- removed link j2n6s300_link_5
- removed link j2n6s300_link_6
- removed link j2n6s300_link_base
- added link gripperMover, mass 0.27621302; collision mesh filename=package://qm_description/meshes/manipulator/z1_GripperMover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 scale=1 1 1; visual mesh filename=package://qm_description/meshes/manipulator/z1_GripperMover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 scale=1 1 1
- added link gripperStator, mass 0.52603655; collision mesh filename=package://qm_description/meshes/manipulator/z1_GripperStato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 scale=1 1 1; visual mesh filename=package://qm_description/meshes/manipulator/z1_GripperStato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 scale=1 1 1
- added link link00, mass 0.47247481; collision cylinder length=0.051 radius=0.0325; visual mesh filename=package://qm_description/meshes/manipulator/z1_Link00.stl scale=1 1 1
- added link link01, mass 0.67332551; collision cylinder length=0.102 radius=0.0325; visual mesh filename=package://qm_description/meshes/manipulator/z1_Link01.stl scale=1 1 1
- added link link02, mass 1.19132258; collision cylinder length=0.051 radius=0.0325; collision cylinder length=0.102 radius=0.0325
- added link link03, mass 0.83940874; collision cylinder length=0.059 radius=0.0325; collision cylinder length=0.116 radius=0.02
- added link link04, mass 0.56404563; collision cylinder length=0.067 radius=0.0325; visual mesh filename=package://qm_description/meshes/manipulator/z1_Link04.stl scale=1 1 1
- added link link05, mass 0.38938492; visual mesh filename=package://qm_description/meshes/manipulator/z1_Link05.stl scale=1 1 1
- added link link06, mass 0.28875807; collision cylinder length=0.051 radius=0.0325; visual mesh filename=package://qm_description/meshes/manipulator/z1_Link06.stl scale=1 1 1
- added link world
Joints:
- removed joint j2n6s300_joint_1
- removed joint j2n6s300_joint_2
- removed joint j2n6s300_joint_3
- removed joint j2n6s300_joint_4
- removed joint j2n6s300_joint_5
- removed joint j2n6s300_joint_6
- removed joint j2n6s300_joint_base
- removed joint j2n6s300_joint_end_effector
- removed joint manipulator_joint
- added joint base_static_joint: type fixed, parent world, child base, origin xyz=0 0 0 rpy=0 0 0
- added joint gripperStator: type fixed, parent link06, child gripperStator, origin xyz=0.051 0.0 0.0 rpy=0 0 0
- added joint joint1: type revolute, parent link00, child link01, origin xyz=0 0 0.0585 rpy=0 0 0, axis 0 0 1, limit lower=-2.6179938779914944 upper=2.6179938779914944 effort=30.0 velocity=3.1415
- added joint joint2: type revolute, parent link01, child link02, origin xyz=0 0 0.045 rpy=0 0 0, axis 0 1 0, limit lower=0.0 upper=2.9670597283903604 effort=60.0 velocity=3.1415
- added joint joint3: type revolute, parent link02, child link03, origin xyz=-0.35 0 0 rpy=0 0 0, axis 0 1 0, limit lower=-2.8797932657906435 upper=0.0 effort=30.0 velocity=3.1415
- added joint joint4: type revolute, parent link03, child link04, origin xyz=0.218 0 0.057 rpy=0 0 0, axis 0 1 0, limit lower=-1.5184364492350666 upper=1.5184364492350666 effort=30.0 velocity=3.1415
- added joint joint5: type revolute, parent link04, child link05, origin xyz=0.07 0.0 0.0 rpy=0 0 0, axis 0 0 1, limit lower=-1.3439035240356338 upper=1.3439035240356338 effort=30.0 velocity=3.1415
- added joint joint6: type revolute, parent link05, child link06, origin xyz=0.0492 0.0 0.0 rpy=0 0 0, axis 1 0 0, limit lower=-2.792526803190927 upper=2.792526803190927 effort=30.0 velocity=3.1415
- added joint jointGripper: type revolute, parent gripperStator, child gripperMover, origin xyz=0.049 0.0 0 rpy=0 0 0, axis 0 1 0, limit lower=-1.5707963267948966 upper=0.0 effort=30.0 velocity=3.1415
- added joint trunk_arm_joint: type fixed, parent base, child link00, origin xyz=0.2535 0 0.056 rpy=0 0 0
- joint LF_HFE: limit lower=-1e+22 upper=1e+22 effort=35.278 velocity=20 -> lower=-2.0943951023931953 upper=4.1887902047863905 effort=35.278 velocity=20
- joint LH_HFE: limit lower=-1e+22 upper=1e+22 effort=35.278 velocity=20 -> lower=-2.0943951023931953 upper=4.1887902047863905 effort=35.278 velocity=20
- joint RF_HFE: limit lower=-1e+22 upper=1e+22 effort=35.278 velocity=20 -> lower=-2.0943951023931953 upper=4.1887902047863905 effort=35.278 velocity=20
- joint RH_HFE: limit lower=-1e+22 upper=1e+22 effort=35.278 velocity=20 -> lower=-2.0943951023931953 upper=4.1887902047863905 effort=35.278 velocity=20
