Commit message: Controller correction

File: qm_description/urdf/manipulator/gazebo.xacro (robot description, xacro)
@@ -7,13 +7,13 @@
         </plugin>
     </gazebo>
-    <gazebo reference="link04">
+    <gazebo reference="z1_link_4">
         <self_collide>true</self_collide>
         <material>Gazebo/DarkGrey</material>
     </gazebo>
-    <gazebo reference="link05">
+    <gazebo reference="z1_link_5">
         <self_collide>true</self_collide>
         <material>Gazebo/DarkGrey</material>
     </gazebo>
-    <gazebo reference="link06">
+    <gazebo reference="z1_link_6">
         <self_collide>true</self_collide>
         <material>Gazebo/DarkGrey</material>

File: qm_description/urdf/manipulator/robot.xacro (robot description, xacro)
@@ -10,7 +10,7 @@
         <origin rpy="0 0 0" xyz="0 0 0"/>
         <parent link="world"/>
-        <child link="link00"/>
-    </joint>
-    <link name="link00">
+        <child link="z1_link_0"/>
+    </joint>
+    <link name="z1_link_0">
         <visual>
             <origin rpy="0 0 0" xyz="0 0 0"/>
@@ -35,13 +35,13 @@
         </inertial>
     </link>
-    <joint name="joint1" type="revolute">
+    <joint name="z1_joint_1" type="revolute">
         <origin rpy="0 0 0" xyz="0 0 0.0585"/>
-        <parent link="link00"/>
-        <child link="link01"/>
+        <parent link="z1_link_0"/>
+        <child link="z1_link_1"/>
         <axis xyz="0 0 1"/>
         <dynamics damping="${jointDamping}" friction="${jointFriction}"/>
         <limit effort="${torqueMax}" velocity="${velocityMax}" lower="${joint1_PositionMin}" upper="${joint1_PositionMax}"/>
     </joint>
-    <link name="link01">
+    <link name="z1_link_1">
         <visual>
             <origin rpy="0 0 0" xyz="0 0 0"/>
@@ -60,13 +60,13 @@
         </inertial>
     </link>
-    <joint name="joint2" type="revolute">
+    <joint name="z1_joint_2" type="revolute">
         <origin rpy="0 0 0" xyz="0 0 0.045"/>
-        <parent link="link01"/>
-        <child link="link02"/>
+        <parent link="z1_link_1"/>
+        <child link="z1_link_2"/>
         <axis xyz="0 1 0"/>
         <dynamics damping="${2*jointDamping}" friction="${2*jointFriction}"/>
         <limit effort="${2*torqueMax}" velocity="${velocityMax}" lower="${joint2_PositionMin}" upper="${joint2_PositionMax}"/>
     </joint>
-    <link name="link02">
+    <link name="z1_link_2">
         <visual>
             <origin rpy="0 0 0" xyz="0 0 0"/>
@@ -103,13 +103,13 @@
         </inertial>
     </link>
-    <joint name="joint3" type="revolute">
+    <joint name="z1_joint_3" type="revolute">
         <origin rpy="0 0 0" xyz="-0.35 0 0"/>
-        <parent link="link02"/>
-        <child link="link03"/>
+        <parent link="z1_link_2"/>
+        <child link="z1_link_3"/>
         <axis xyz="0 1 0"/>
         <dynamics damping="${jointDamping}" friction="${jointFriction}"/>
         <limit effort="${torqueMax}" velocity="${velocityMax}" lower="${joint3_PositionMin}" upper="${joint3_PositionMax}"/>
     </joint>
-    <link name="link03">
+    <link name="z1_link_3">
         <visual>
             <origin rpy="0 0 0" xyz="0 0 0"/>
@@ -140,13 +140,13 @@
         </inertial>
     </link>
-    <joint name="joint4" type="revolute">
+    <joint name="z1_joint_4" type="revolute">
         <origin rpy="0 0 0" xyz="0.218 0 0.057"/>
-        <parent link="link03"/>
-        <child link="link04"/>
+        <parent link="z1_link_3"/>
+        <child link="z1_link_4"/>
         <axis xyz="0 1 0"/>
         <dynamics damping="${jointDamping}" friction="${jointFriction}"/>
         <limit effort="${torqueMax}" velocity="${velocityMax}" lower="${joint4_PositionMin}" upper="${joint4_PositionMax}"/>
     </joint>
-    <link name="link04">
+    <link name="z1_link_4">
         <visual>
             <origin rpy="0 0 0" xyz="0 0 0"/>
@@ -171,13 +171,13 @@
         </inertial>
     </link>
-    <joint name="joint5" type="revolute">
+    <joint name="z1_joint_5" type="revolute">
         <origin rpy="0 0 0" xyz="0.07 0.0 0.0"/>
-        <parent link="link04"/>
-        <child link="link05"/>
+        <parent link="z1_link_4"/>
+        <child link="z1_link_5"/>
         <axis xyz="0 0 1"/>
         <dynamics damping="${jointDamping}" friction="${jointFriction}"/>
         <limit effort="${torqueMax}" velocity="${velocityMax}" lower="${joint5_PositionMin}" upper="${joint5_PositionMax}"/>
     </joint>
-    <link name="link05">
+    <link name="z1_link_5">
         <visual>
             <origin rpy="0 0 0" xyz="0 0 0"/>
@@ -196,13 +196,13 @@
         </inertial>
     </link>
-    <joint name="joint6" type="revolute">
+    <joint name="z1_joint_6" type="revolute">
         <origin rpy="0 0 0" xyz="0.0492 0.0 0.0"/>
-        <parent link="link05"/>
-        <child link="link06"/>
+        <parent link="z1_link_5"/>
+        <child link="z1_link_6"/>
         <axis xyz="1 0 0"/>
         <dynamics damping="${jointDamping}" friction="${jointFriction}"/>
         <limit effort="${torqueMax}" velocity="${velocityMax}" lower="${joint6_PositionMin}" upper="${joint6_PositionMax}"/>
     </joint>
-    <link name="link06">
+    <link name="z1_link_6">
         <visual>
             <origin rpy="0 0 0" xyz="0 0 0"/>
@@ -230,5 +230,5 @@
         <joint name="gripperStator" type="fixed">
             <origin rpy="0 0 0" xyz="0.051 0.0 0.0"/>
-            <parent link="link06"/>
+            <parent link="z1_link_6"/>
             <child link="gripperStator"/>
         </joint>
@@ -254,5 +254,5 @@
             </inertial>
         </link>
-        <joint name="jointGripper" type="revolute">
+        <joint name="z1_joint_Gripper" type="revolute">
             <origin rpy="0 0 0" xyz="0.049 0.0 0"/>
             <parent link="gripperStator"/>

File: qm_description/urdf/manipulator/transmission.xacro (robot description, xacro)
@@ -4,5 +4,5 @@
         <transmission name="z1_joint_${name}_trans">
             <type>transmission_interface/SimpleTransmission</type>
-            <joint name="joint${name}">
+            <joint name="z1_joint_${name}">
                 <hardwareInterface>hardware_interface/EffortJointInterface</hardwareInterface>
             </joint>

File: qm_description/urdf/quadruped_manipulator/gazebo.xacro (robot description, xacro)
@@ -136,30 +136,30 @@
     </gazebo>
     <!-- Z1 arm -->
-     <gazebo reference="link00">
+     <gazebo reference="z1_link_0">
         <material>Gazebo/Grey</material>
     </gazebo>
-     <gazebo reference="link01">
+     <gazebo reference="z1_link_1">
         <material>Gazebo/Grey</material>
         <provideFeedback>true</provideFeedback>
     </gazebo>
-    <gazebo reference="link02">
+    <gazebo reference="z1_link_2">
         <material>Gazebo/Grey</material>
         <provideFeedback>true</provideFeedback>
     </gazebo>
-    <gazebo reference="link03">
+    <gazebo reference="z1_link_3">
         <material>Gazebo/Grey</material>
         <provideFeedback>true</provideFeedback>
     </gazebo>
-    <gazebo reference="link04">
+    <gazebo reference="z1_link_4">
         <self_collide>true</self_collide>
         <material>Gazebo/Grey</material>
         <provideFeedback>true</provideFeedback>
     </gazebo>
-    <gazebo reference="link05">
+    <gazebo reference="z1_link_5">
         <self_collide>true</self_collide>
         <material>Gazebo/Grey</material>
         <provideFeedback>true</provideFeedback>
     </gazebo>
-    <gazebo reference="link06">
+    <gazebo reference="z1_link_6">
         <self_collide>true</self_collide>
         <material>Gazebo/Grey</material>

File: qm_description/urdf/quadruped_manipulator/robot.urdf (robot description, URDF)
Before this commit: robot qm, 28 links, 27 joints
Links:
- removed link link00
- removed link link01
- removed link link02
- removed link link03
- removed link link04
- removed link link05
- removed link link06
- added link z1_link_0, mass 0.47247481; collision cylinder length=0.051 radius=0.0325; visual mesh filename=package://qm_description/meshes/manipulator/z1_Link00.stl scale=1 1 1
- added link z1_link_1, mass 0.67332551; collision cylinder length=0.102 radius=0.0325; visual mesh filename=package://qm_description/meshes/manipulator/z1_Link01.stl scale=1 1 1
- added link z1_link_2, mass 1.19132258; collision cylinder length=0.051 radius=0.0325; collision cylinder length=0.102 radius=0.0325
- added link z1_link_3, mass 0.83940874; collision cylinder length=0.059 radius=0.0325; collision cylinder length=0.116 radius=0.02
- added link z1_link_4, mass 0.56404563; collision cylinder length=0.067 radius=0.0325; visual mesh filename=package://qm_description/meshes/manipulator/z1_Link04.stl scale=1 1 1
- added link z1_link_5, mass 0.38938492; visual mesh filename=package://qm_description/meshes/manipulator/z1_Link05.stl scale=1 1 1
- added link z1_link_6, mass 0.28875807; collision cylinder length=0.051 radius=0.0325; visual mesh filename=package://qm_description/meshes/manipulator/z1_Link06.stl scale=1 1 1
Joints:
- removed joint joint1
- removed joint joint2
- removed joint joint3
- removed joint joint4
- removed joint joint5
- removed joint joint6
- removed joint jointGripper
- added joint z1_joint_1: type revolute, parent z1_link_0, child z1_link_1, origin xyz=0 0 0.0585 rpy=0 0 0, axis 0 0 1, limit lower=-2.6179938779914944 upper=2.6179938779914944 effort=30.0 velocity=3.1415
- added joint z1_joint_2: type revolute, parent z1_link_1, child z1_link_2, origin xyz=0 0 0.045 rpy=0 0 0, axis 0 1 0, limit lower=0.0 upper=2.9670597283903604 effort=60.0 velocity=3.1415
- added joint z1_joint_3: type revolute, parent z1_link_2, child z1_link_3, origin xyz=-0.35 0 0 rpy=0 0 0, axis 0 1 0, limit lower=-2.8797932657906435 upper=0.0 effort=30.0 velocity=3.1415
- added joint z1_joint_4: type revolute, parent z1_link_3, child z1_link_4, origin xyz=0.218 0 0.057 rpy=0 0 0, axis 0 1 0, limit lower=-1.5184364492350666 upper=1.5184364492350666 effort=30.0 velocity=3.1415
- added joint z1_joint_5: type revolute, parent z1_link_4, child z1_link_5, origin xyz=0.07 0.0 0.0 rpy=0 0 0, axis 0 0 1, limit lower=-1.3439035240356338 upper=1.3439035240356338 effort=30.0 velocity=3.1415
- added joint z1_joint_6: type revolute, parent z1_link_5, child z1_link_6, origin xyz=0.0492 0.0 0.0 rpy=0 0 0, axis 1 0 0, limit lower=-2.792526803190927 upper=2.792526803190927 effort=30.0 velocity=3.1415
- added joint z1_joint_Gripper: type revolute, parent gripperStator, child gripperMover, origin xyz=0.049 0.0 0 rpy=0 0 0, axis 0 1 0, limit lower=-1.5707963267948966 upper=0.0 effort=30.0 velocity=3.1415
- joint gripperStator: parent link06 -> z1_link_6
- joint manipulator_joint: child link00 -> z1_link_0

File: qm_description/urdf/quadruped_manipulator/robot.xacro (robot description, xacro)
@@ -11,4 +11,13 @@
     <xacro:include filename="$(find qm_description)/urdf/manipulator/transmission.xacro"/>
     <xacro:arg name="UnitreeGripper" default="true"/>
+  <!-- Debug mode will hung up the robot, use "true" or "false" to switch it. -->
+    <xacro:if value="$(arg DEBUG)">
+        <link name="world"/>
+        <joint name="base_static_joint" type="fixed">
+            <origin rpy="0 0 0" xyz="0 0 0"/>
+            <parent link="world"/>
+            <child link="base"/>
+        </joint>
+    </xacro:if>
      <!-- Aliengo robot -->
      <link name="base">
@@ -53,7 +62,7 @@
         <origin rpy="${arm_offset_r} ${arm_offset_p} ${arm_offset_yaw}" xyz="${arm_offset_x} ${arm_offset_y} ${arm_offset_z}"/>
         <parent link="base"/>
-        <child link="link00"/>
-    </joint>
-    <link name="link00">
+        <child link="z1_link_0"/>
+    </joint>
+    <link name="z1_link_0">
         <visual>
             <origin rpy="0 0 0" xyz="0 0 0"/>
@@ -78,8 +87,8 @@
         </inertial>
     </link>
-   <joint name="joint1" type="revolute">
+   <joint name="z1_joint_1" type="revolute">
         <origin rpy="0 0 0" xyz="0 0 0.0585"/>
-        <parent link="link00"/>
-        <child link="link01"/>
+        <parent link="z1_link_0"/>
+        <child link="z1_link_1"/>
         <axis xyz="0 0 1"/>
         <dynamics damping="${jointDamping}" friction="${jointFriction}"/>
@@ -90,9 +99,9 @@
         <plugin filename="libgazebo_ros_ft_sensor.so" name="ft_sensor">
         <updateRate>30.0</updateRate>
-        <topicName>joint1_ft_sensor_topic</topicName>
-        <jointName>joint1</jointName>
-        </plugin>
-    </gazebo>
-    <link name="link01">
+        <topicName>z1_joint_1_ft_sensor_topic</topicName>
+        <jointName>z1_joint_1</jointName>
+        </plugin>
+    </gazebo>
+    <link name="z1_link_1">
         <visual>
             <origin rpy="0 0 0" xyz="0 0 0"/>
@@ -117,8 +126,8 @@
         </inertial>
     </link>
-    <joint name="joint2" type="revolute">
+    <joint name="z1_joint_2" type="revolute">
         <origin rpy="0 0 0" xyz="0 0 0.045"/>
-        <parent link="link01"/>
-        <child link="link02"/>
+        <parent link="z1_link_1"/>
+        <child link="z1_link_2"/>
         <axis xyz="0 1 0"/>
         <dynamics damping="${2*jointDamping}" friction="${2*jointFriction}"/>
@@ -129,9 +138,9 @@
         <plugin filename="libgazebo_ros_ft_sensor.so" name="ft_sensor">
         <updateRate>30.0</updateRate>
-        <topicName>joint2_ft_sensor_topic</topicName>
-        <jointName>joint2</jointName>
-        </plugin>
-    </gazebo>
-    <link name="link02">
+        <topicName>z1_joint_2_ft_sensor_topic</topicName>
+        <jointName>z1_joint_2</jointName>
+        </plugin>
+    </gazebo>
+    <link name="z1_link_2">
         <visual>
             <origin rpy="0 0 0" xyz="0 0 0"/>
@@ -168,8 +177,8 @@
         </inertial>
     </link>
-    <joint name="joint3" type="revolute">
+    <joint name="z1_joint_3" type="revolute">
         <origin rpy="0 0 0" xyz="-0.35 0 0"/>
-        <parent link="link02"/>
-        <child link="link03"/>
+        <parent link="z1_link_2"/>
+        <child link="z1_link_3"/>
         <axis xyz="0 1 0"/>
         <dynamics damping="${jointDamping}" friction="${jointFriction}"/>
@@ -180,9 +189,9 @@
         <plugin filename="libgazebo_ros_ft_sensor.so" name="ft_sensor">
         <updateRate>30.0</updateRate>
-        <topicName>joint3_ft_sensor_topic</topicName>
-        <jointName>joint3</jointName>
-        </plugin>
-    </gazebo>
-    <link name="link03">
+        <topicName>z1_joint_3_ft_sensor_topic</topicName>
+        <jointName>z1_joint_3</jointName>
+        </plugin>
+    </gazebo>
+    <link name="z1_link_3">
         <visual>
             <origin rpy="0 0 0" xyz="0 0 0"/>
@@ -213,8 +222,8 @@
         </inertial>
     </link>
-    <joint name="joint4" type="revolute">
+    <joint name="z1_joint_4" type="revolute">
         <origin rpy="0 0 0" xyz="0.218 0 0.057"/>
-        <parent link="link03"/>
-        <child link="link04"/>
+        <parent link="z1_link_3"/>
+        <child link="z1_link_4"/>
         <axis xyz="0 1 0"/>
         <dynamics damping="${jointDamping}" friction="${jointFriction}"/>
@@ -225,9 +234,9 @@
         <plugin filename="libgazebo_ros_ft_sensor.so" name="ft_sensor">
         <updateRate>30.0</updateRate>
-        <topicName>joint4_ft_sensor_topic</topicName>
-        <jointName>joint4</jointName>
-        </plugin>
-    </gazebo>
-    <link name="link04">
+        <topicName>z1_joint_4_ft_sensor_topic</topicName>
+        <jointName>z1_joint_4</jointName>
+        </plugin>
+    </gazebo>
+    <link name="z1_link_4">
         <visual>
             <origin rpy="0 0 0" xyz="0 0 0"/>
@@ -252,8 +261,8 @@
         </inertial>
     </link>
-    <joint name="joint5" type="revolute">
+    <joint name="z1_joint_5" type="revolute">
         <origin rpy="0 0 0" xyz="0.07 0.0 0.0"/>
-        <parent link="link04"/>
-        <child link="link05"/>
+        <parent link="z1_link_4"/>
+        <child link="z1_link_5"/>
         <axis xyz="0 0 1"/>
         <dynamics damping="${jointDamping}" friction="${jointFriction}"/>
@@ -264,9 +273,9 @@
         <plugin filename="libgazebo_ros_ft_sensor.so" name="ft_sensor">
         <updateRate>30.0</updateRate>
-        <topicName>joint5_ft_sensor_topic</topicName>
-        <jointName>joint5</jointName>
-        </plugin>
-    </gazebo>
-    <link name="link05">
+        <topicName>z1_joint_5_ft_sensor_topic</topicName>
+        <jointName>z1_joint_5</jointName>
+        </plugin>
+    </gazebo>
+    <link name="z1_link_5">
         <visual>
             <origin rpy="0 0 0" xyz="0 0 0"/>
@@ -285,8 +294,8 @@
         </inertial>
     </link>
-    <joint name="joint6" type="revolute">
+    <joint name="z1_joint_6" type="revolute">
         <origin rpy="0 0 0" xyz="0.0492 0.0 0.0"/>
-        <parent link="link05"/>
-        <child link="link06"/>
+        <parent link="z1_link_5"/>
+        <child link="z1_link_6"/>
         <axis xyz="1 0 0"/>
         <dynamics damping="${jointDamping}" friction="${jointFriction}"/>
@@ -297,9 +306,9 @@
         <plugin filename="libgazebo_ros_ft_sensor.so" name="ft_sensor">
         <updateRate>30.0</updateRate>
-        <topicName>joint6_ft_sensor_topic</topicName>
-        <jointName>joint6</jointName>
-        </plugin>
-    </gazebo>
-    <link name="link06">
+        <topicName>z1_joint_6_ft_sensor_topic</topicName>
+        <jointName>z1_joint_6</jointName>
+        </plugin>
+    </gazebo>
+    <link name="z1_link_6">
         <visual>
             <origin rpy="0 0 0" xyz="0 0 0"/>
@@ -327,5 +336,5 @@
         <joint name="gripperStator" type="fixed">
             <origin rpy="0 0 0" xyz="0.051 0.0 0.0"/>
-            <parent link="link06"/>
+            <parent link="z1_link_6"/>
             <child link="gripperStator"/>
         </joint>
@@ -352,5 +361,5 @@
             </inertial>
         </link>
-        <joint name="jointGripper" type="revolute">
+        <joint name="z1_joint_Gripper" type="revolute">
             <origin rpy="0 0 0" xyz="0.049 0.0 0"/>
             <parent link="gripperStator"/>
