Commit message: Debugging

File: qm_description/urdf/quadruped/aliengo/const.xacro (robot description, xacro)
@@ -36,6 +36,6 @@
     <xacro:property name="hip_velocity_max" value="20"/>
     <xacro:property name="hip_torque_max" value="35.278"/>
-    <xacro:property name="thigh_max" value="${240*pi/180.0}"/>     <!-- 1e22 -->
-    <xacro:property name="thigh_min" value="${-120*pi/180.0}"/>    <!-- -1e22 -->
+    <xacro:property name="thigh_max" value="1e22"/>     <!-- 240*pi/180.0 -->
+    <xacro:property name="thigh_min" value="-1e22"/>    <!-- ${-120*pi/180.0} -->
     <xacro:property name="thigh_velocity_max" value="20"/>
     <xacro:property name="thigh_torque_max" value="35.278"/>
