Commit message: :tada: START: Initial commit

File: qm_description/urdf/doors/door_pull.xacro (robot description, xacro)
@@ -5,5 +5,5 @@
     <parent link="world"/>
     <child link="frame"/>
-    <origin rpy= "0 0 1.5708" xyz="-0.075 0.425 0"/>
+    <origin rpy= "0 0 -1.5708" xyz="0.075 -0.425 0"/>
   </joint>
 <link name="frame">
@@ -37,8 +37,8 @@
     <inertial>
       <origin rpy="0 0 0" xyz="0 0 0"/>
-      <mass value="0.1"/>
-      <inertia ixx="0.030386862790" 	ixy="0.000000000330"	ixz="-0.000000216760"
-					iyy="0.035534743650" 	iyz="-0.000000000060"
-								izz="0.005184277950"/>
+      <mass value="20"/>
+      <inertia ixx="6.67" 	ixy="0"	ixz="0"
+					      iyy="2.69" 	iyz="0"
+								izz="6.4"/>
     </inertial>
     <visual>
@@ -64,5 +64,5 @@
     <parent link="frame"/>
     <child link="door"/>
-    <dynamics damping="0.2" friction="0.000001"/>
+    <dynamics damping="0.01" friction="0.0001"/>
     <origin xyz="0 0 0"/>
     <axis xyz="0 0 1"/>
@@ -72,6 +72,6 @@
     <inertial>
       <origin rpy="0 0 0" xyz="0 0 0"/>
-      <mass value="5.0"/>
-      <inertia ixx="0.01" ixy="0" ixz="0" iyy="0.01" iyz="0" izz="0.01"/>
+      <mass value="0.3"/>
+      <inertia ixx="0.001" ixy="0" ixz="0" iyy="0.001" iyz="0" izz="0.001"/>
     </inertial>
     <visual>
@@ -103,7 +103,7 @@
   <gazebo reference="joint_door_lever">
     <implicitSpringDamper>true</implicitSpringDamper>
-    <spring_stiffness>10000</spring_stiffness>
+    <spring_stiffness>500</spring_stiffness>
     <spring_reference>0.0</spring_reference>
-    <damping>10.0</damping>
+    <damping>0.1</damping>
   </gazebo>
   </joint>

File: qm_description/urdf/doors/door_push.xacro (robot description, xacro)
@@ -37,8 +37,8 @@
     <inertial>
       <origin rpy="0 0 0" xyz="0 0 0"/>
-      <mass value="0.1"/>
-      <inertia ixx="0.030386862790" 	ixy="0.000000000330"	ixz="-0.000000216760"
-					iyy="0.035534743650" 	iyz="-0.000000000060"
-								izz="0.005184277950"/>
+      <mass value="20"/>
+      <inertia ixx="6.67" 	ixy="0"	ixz="0"
+					      iyy="2.69" 	iyz="0"
+								izz="6.4"/>
     </inertial>
     <visual>
@@ -64,5 +64,5 @@
     <parent link="frame"/>
     <child link="door"/>
-    <dynamics damping="0.2" friction="0.000001"/>
+    <dynamics damping="0.01" friction="0.0001"/>
     <origin xyz="0 0 0"/>
     <axis xyz="0 0 1"/>
@@ -72,6 +72,6 @@
     <inertial>
       <origin rpy="0 0 0" xyz="0 0 0"/>
-      <mass value="5.0"/>
-      <inertia ixx="0.01" ixy="0" ixz="0" iyy="0.01" iyz="0" izz="0.01"/>
+      <mass value="0.3"/>
+      <inertia ixx="0.001" ixy="0" ixz="0" iyy="0.001" iyz="0" izz="0.001"/>
     </inertial>
     <visual>
@@ -103,7 +103,7 @@
   <gazebo reference="joint_door_lever">
     <implicitSpringDamper>true</implicitSpringDamper>
-    <spring_stiffness>10000</spring_stiffness>
+    <spring_stiffness>500</spring_stiffness>
     <spring_reference>0.0</spring_reference>
-    <damping>10.0</damping>
+    <damping>0.1</damping>
   </gazebo>
   </joint>

File: qm_description/urdf/pallets/pallet1.xacro (robot description, xacro)
@@ -14,4 +14,12 @@
         <mesh filename="package://qm_description/meshes/pallets/Pallet13cm.stl" scale="0.001 0.001 0.001"/>
       </geometry>
+      <surface>
+        <friction>
+            <ode>
+                <mu>0.7</mu>        <!-- Primary friction coefficient -->
+                <mu2>0.7</mu2>      <!-- Secondary friction coefficient -->
+            </ode>
+        </friction>
+      </surface>
     </collision>
     <inertial>

File: qm_description/urdf/pallets/pallet2.xacro (robot description, xacro)
@@ -14,4 +14,12 @@
         <mesh filename="package://qm_description/meshes/pallets/Pallet15cm.stl" scale="0.001 0.001 0.001"/>
       </geometry>
+      <surface>
+        <friction>
+            <ode>
+                <mu>0.7</mu>        <!-- Primary friction coefficient -->
+                <mu2>0.7</mu2>      <!-- Secondary friction coefficient -->
+            </ode>
+        </friction>
+      </surface>
     </collision>
     <inertial>

File: qm_description/urdf/pallets/pallet3.xacro (robot description, xacro)
@@ -14,4 +14,12 @@
         <mesh filename="package://qm_description/meshes/pallets/Pallet18cm.stl" scale="0.001 0.001 0.001"/>
       </geometry>
+      <surface>
+        <friction>
+            <ode>
+                <mu>0.7</mu>        <!-- Primary friction coefficient -->
+                <mu2>0.7</mu2>      <!-- Secondary friction coefficient -->
+            </ode>
+        </friction>
+      </surface>
     </collision>
     <inertial>

File: qm_description/urdf/pallets/pallet4.xacro (robot description, xacro)
@@ -14,4 +14,12 @@
         <mesh filename="package://qm_description/meshes/pallets/Pallet20cm.stl" scale="0.001 0.001 0.001"/>
       </geometry>
+      <surface>
+        <friction>
+            <ode>
+                <mu>0.7</mu>        <!-- Primary friction coefficient -->
+                <mu2>0.7</mu2>      <!-- Secondary friction coefficient -->
+            </ode>
+        </friction>
+      </surface>
     </collision>
     <inertial>

File: qm_description/urdf/quadruped/common/leg.xacro (robot description, xacro)
@@ -120,4 +120,12 @@
                     <box size="${calf_length} ${calf_width} ${calf_height}"/>
                 </geometry>
+                <surface>
+                    <friction>
+                        <ode>
+                            <mu>1</mu>        <!-- Primary friction coefficient -->
+                            <mu2>1</mu2>      <!-- Secondary friction coefficient -->
+                        </ode>
+                    </friction>
+                </surface>
             </collision>
             <inertial>
@@ -151,6 +159,6 @@
                     <friction>
                         <ode>
-                            <mu>0.7</mu>        <!-- Primary friction coefficient -->
-                            <mu2>0.7</mu2>      <!-- Secondary friction coefficient -->
+                            <mu>1</mu>        <!-- Primary friction coefficient -->
+                            <mu2>1</mu2>      <!-- Secondary friction coefficient -->
                         </ode>
                     </friction>

File: qm_description/urdf/quadruped_manipulator/robot.xacro (robot description, xacro)
@@ -11,4 +11,5 @@
     <xacro:include filename="$(find qm_description)/urdf/manipulator/transmission.xacro"/>
     <xacro:include filename="$(find qm_description)/urdf/quadruped_manipulator/camera.xacro"/>
+    <xacro:include filename="$(find qm_description)/urdf/quadruped_manipulator/camera2.xacro"/>
     <xacro:arg name="UnitreeGripper" default="true"/>
   <!-- Debug mode will hung up the robot, use "true" or "false" to switch it. -->
@@ -44,4 +45,8 @@
         </inertial>
     </link>
+    <!-- D435 IntelRealSense Camera -->
+    <xacro:sensor_d435 parent="base" name="camera2" use_nominal_extrinsics="true">
+        <origin xyz="0.32 0.01 -0.035" rpy="0 0 0"/>
+    </xacro:sensor_d435>
     <!-- IMU -->
     <xacro:IMU connected_to="base" imu_name="unitree_imu" xyz="0. 0. 0." rpy="0. 0. 0."/>
@@ -482,4 +487,5 @@
             </inertial>
         </link>
+        <!-- TODO Change to revolute once controller is programmed -->
         <joint name="z1_joint_Gripper" type="revolute">
             <origin rpy="0 0 0" xyz="0.049 0.0 0"/>
@@ -528,5 +534,5 @@
         </link>
         <link name="z1_end_effector">
-            <visual>
+            <!-- <visual>
                 <geometry>
                     <sphere radius="0.01"/>
@@ -547,5 +553,5 @@
                     </contact>
                 </surface>
-            </collision>
+            </collision> -->
         </link>
         <joint name="z1_joint_end_effector" type="fixed">

File: qm_description/urdf/sar/ball10.xacro (robot description, xacro)
@@ -1,31 +1,25 @@
 <?xml version="1.0"?>
-<robot name="sar" xmlns:xacro="http://www.ros.org/wiki/xacro">
-  <link name="sar_link">
+<robot name="sphere10" xmlns:xacro="http://www.ros.org/wiki/xacro">
+  <link name="sphere10_link">
     <visual>
       <geometry>
-        <mesh filename="package://qm_description/meshes/sar/TerrainMobile.stl" scale="0.001 0.001 0.001"/>
+        <mesh filename="package://qm_description/meshes/sar/Sphere10.stl" scale="0.001 0.001 0.001"/>
       </geometry>
-      <material name="ocher">
-          <color rgba="0.949 0.890 0.722 1"/>
+      <material name="gray">
+          <color rgba="0.435 0.4 0.329 1"/>
       </material>
     </visual>
     <collision>
       <geometry>
-        <mesh filename="package://qm_description/meshes/sar/TerrainMobile.stl" scale="0.001 0.001 0.001"/>
+        <mesh filename="package://qm_description/meshes/sar/Sphere10.stl" scale="0.001 0.001 0.001"/>
       </geometry>
     </collision>
     <inertial>
-      <mass value="1.0"/>
-      <inertia ixx="0.1" ixy="0.0" ixz="0.0" iyy="0.1" iyz="0.0" izz="0.1"/>
+      <mass value="3.77"/>
+      <inertia ixx="0.01508" ixy="0.0" ixz="0.0" iyy="0.01508" iyz="0.0" izz="0.01508"/>
     </inertial>
   </link>
-  <gazebo reference="sar_link">
-    <material>Gazebo/Wood</material>
+  <gazebo reference="sphere10_link">
+    <material>Gazebo/Grey</material>
   </gazebo>
-  <!-- Wall fixed to the world-->
-  <link name="world"/>
-  <joint name="base_link_fixed" type="fixed">
-    <parent link="world"/>
-    <child link="sar_link"/>
-  </joint>
 </robot>

File: qm_description/urdf/sar/ball15.xacro (robot description, xacro)
@@ -1,31 +1,25 @@
 <?xml version="1.0"?>
-<robot name="sar" xmlns:xacro="http://www.ros.org/wiki/xacro">
-  <link name="sar_link">
+<robot name="sphere15" xmlns:xacro="http://www.ros.org/wiki/xacro">
+  <link name="sphere15_link">
     <visual>
       <geometry>
-        <mesh filename="package://qm_description/meshes/sar/TerrainMobile.stl" scale="0.001 0.001 0.001"/>
+        <mesh filename="package://qm_description/meshes/sar/Sphere15.stl" scale="0.001 0.001 0.001"/>
       </geometry>
-      <material name="ocher">
-          <color rgba="0.949 0.890 0.722 1"/>
+      <material name="gray">
+          <color rgba="0.435 0.4 0.329 1"/>
       </material>
     </visual>
     <collision>
       <geometry>
-        <mesh filename="package://qm_description/meshes/sar/TerrainMobile.stl" scale="0.001 0.001 0.001"/>
+        <mesh filename="package://qm_description/meshes/sar/Sphere15.stl" scale="0.001 0.001 0.001"/>
       </geometry>
     </collision>
     <inertial>
-      <mass value="1.0"/>
-      <inertia ixx="0.1" ixy="0.0" ixz="0.0" iyy="0.1" iyz="0.0" izz="0.1"/>
+      <mass value="12.7"/>
+      <inertia ixx="0.1143" ixy="0.0" ixz="0.0" iyy="0.1143" iyz="0.0" izz="0.1143"/>
     </inertial>
   </link>
-  <gazebo reference="sar_link">
-    <material>Gazebo/Wood</material>
+  <gazebo reference="sphere15_link">
+    <material>Gazebo/Grey</material>
   </gazebo>
-  <!-- Wall fixed to the world-->
-  <link name="world"/>
-  <joint name="base_link_fixed" type="fixed">
-    <parent link="world"/>
-    <child link="sar_link"/>
-  </joint>
 </robot>

File: qm_description/urdf/sar/plate.xacro (robot description, xacro)
@@ -1,31 +1,26 @@
 <?xml version="1.0"?>
-<robot name="sar" xmlns:xacro="http://www.ros.org/wiki/xacro">
-  <link name="sar_link">
+<robot name="plate" xmlns:xacro="http://www.ros.org/wiki/xacro">
+  <link name="plate_link">
     <visual>
       <geometry>
-        <mesh filename="package://qm_description/meshes/sar/TerrainMobile.stl" scale="0.001 0.001 0.001"/>
+        <mesh filename="package://qm_description/meshes/sar/Plate.stl" scale="0.005 0.001 0.001"/>
       </geometry>
-      <material name="ocher">
-          <color rgba="0.949 0.890 0.722 1"/>
+      <material name="brown">
+          <color rgba="0.612 0.447 0.114 1"/>
       </material>
     </visual>
     <collision>
       <geometry>
-        <mesh filename="package://qm_description/meshes/sar/TerrainMobile.stl" scale="0.001 0.001 0.001"/>
+        <mesh filename="package://qm_description/meshes/sar/Plate.stl" scale="0.005 0.001 0.001"/>
       </geometry>
     </collision>
     <inertial>
-      <mass value="1.0"/>
-      <inertia ixx="0.1" ixy="0.0" ixz="0.0" iyy="0.1" iyz="0.0" izz="0.1"/>
+      <origin xyz="-0.5 0 -0.5" rpy="0 0 0"/>
+      <mass value="10"/>
+      <inertia ixx="0.8354" ixy="0.0" ixz="0.0" iyy="1.667" iyz="0.0" izz="0.8354"/>
     </inertial>
   </link>
-  <gazebo reference="sar_link">
+  <gazebo reference="plate_link">
     <material>Gazebo/Wood</material>
   </gazebo>
-  <!-- Wall fixed to the world-->
-  <link name="world"/>
-  <joint name="base_link_fixed" type="fixed">
-    <parent link="world"/>
-    <child link="sar_link"/>
-  </joint>
 </robot>

File: qm_description/urdf/sar/rod.xacro (robot description, xacro)
@@ -1,31 +1,26 @@
 <?xml version="1.0"?>
-<robot name="sar" xmlns:xacro="http://www.ros.org/wiki/xacro">
-  <link name="sar_link">
+<robot name="rod" xmlns:xacro="http://www.ros.org/wiki/xacro">
+  <link name="rod_link">
     <visual>
       <geometry>
-        <mesh filename="package://qm_description/meshes/sar/TerrainMobile.stl" scale="0.001 0.001 0.001"/>
+        <mesh filename="package://qm_description/meshes/sar/Stick.stl" scale="0.001 0.001 0.001"/>
       </geometry>
-      <material name="ocher">
-          <color rgba="0.949 0.890 0.722 1"/>
+      <material name="brown">
+          <color rgba="0.462 0.345 0.129 1"/>
       </material>
     </visual>
     <collision>
       <geometry>
-        <mesh filename="package://qm_description/meshes/sar/TerrainMobile.stl" scale="0.001 0.001 0.001"/>
+        <mesh filename="package://qm_description/meshes/sar/Stick.stl" scale="0.001 0.001 0.001"/>
       </geometry>
     </collision>
     <inertial>
-      <mass value="1.0"/>
-      <inertia ixx="0.1" ixy="0.0" ixz="0.0" iyy="0.1" iyz="0.0" izz="0.1"/>
+      <origin xyz="0.5 0 0" rpy="0 0 0"/>
+      <mass value="3.0"/>
+      <inertia ixx="0.000375" ixy="0.0" ixz="0.0" iyy="0.25185" iyz="0.0" izz="0.25185"/>
     </inertial>
   </link>
-  <gazebo reference="sar_link">
-    <material>Gazebo/Wood</material>
+  <gazebo reference="rod_link">
+    <material>Gazebo/WoodPallet</material>
   </gazebo>
-  <!-- Wall fixed to the world-->
-  <link name="world"/>
-  <joint name="base_link_fixed" type="fixed">
-    <parent link="world"/>
-    <child link="sar_link"/>
-  </joint>
 </robot>

File: qm_description/urdf/stairs/stairs.xacro (robot description, xacro)
@@ -16,6 +16,6 @@
     <xacro:property name="s2_offset_z" value="${s1_offset_z + s1_height * s1_quantity}"/>
     <xacro:property name="s3_quantity" value="10"/>
-    <xacro:property name="s3_height" value="-0.05"/>
-    <xacro:property name="s3_depth" value="0.1"/>
+    <xacro:property name="s3_height" value="-0.08"/>
+    <xacro:property name="s3_depth" value="0.15"/>
     <xacro:property name="s3_width" value="1.5"/>
     <xacro:property name="s3_offset_x" value="${s2_offset_x + s2_length*cos(s2_angle*pi/180)}"/>
